File: KiCad5/Hardware_NanoPi_v4/WiRoc_NanoPi_v1.kicad_pcb (KiCad board)
At the start: 2 copper layers, 47 x 68.3 mm, 125 parts, among them J1 Conn_01x02, J2 USB_Power_02x02, J3 Serial, J4 USB_Host_Data_02x02, J6 HAT_Conn_DBG, J7 NanoPIAir, J8 USB_Host_Data_02x02, J9 Conn_Coaxial, SW1 SW_SPST, U1 DRF1268DS, U2 OLED, U3 AXP209, U4 LP6226_SY7208, U5 SY6280, U6 BatteryPadM, U7 BatteryPadP

Commit message: etc
Parts:
- removed D4, D5: LED, Diode_SMD:D_0603_1608Metric
- removed the REF** at (72.5, 106.7)
- removed the REF** at (78.2, 106.7)
- removed the REF** at (73.3, 91.2)
- removed the REF** at (71.9, 95.9)
- removed the REF** at (90.7, 75.2)
- removed the REF** at (69.7, 95.9)
- removed the REF** at (67.7, 95.9)
- removed the REF** at (63.1, 93.0)
- removed the REF** at (63.1, 90.6)
- removed the REF** at (84.8, 106.4)
- removed the REF** at (74.0, 83.8)
- removed the REF** at (77.3, 83.6)
- removed the REF** at (77.3, 84.8)
- removed the REF** at (73.2, 88.0)
- removed the REF** at (89.5, 69.7)
- removed the REF** at (74.4, 88.0)
- removed the REF** at (73.3, 93.3)
- removed the REF** at (89.4, 75.9)
- removed the REF** at (74.9, 93.3)
- removed the REF** at (64.2, 83.3)
- removed the REF** at (74.3, 86.5)
- removed the REF** at (77.3, 86.2)
- removed the REF** at (74.3, 85.1)
- removed the REF** at (78.9, 95.6)
- added C16: 1uF, Capacitor_SMD:C_0603_1608Metric, F.Cu at (87.0, 75.5)
- added C17: 47uF, Capacitor_SMD:C_1210_3225Metric, F.Cu at (92.1, 70.6)
- added C18: 4.7uF, Capacitor_SMD:C_0603_1608Metric, F.Cu at (86.4, 70.4)
- added D1: LED_DUAL_ACCA, WiRoc:LED_Dual_1.7_1.6, F.Cu at (92.0, 61.9)
- added R6: 1K, Resistor_SMD:R_0603_1608Metric, F.Cu at (92.0, 64.1)
- added REF**: VIA-0.6mm, WiRoc:VIA-0.6mm, F.Cu at (78.3, 103.5)
- added REF**: VIA-0.6mm, WiRoc:VIA-0.6mm, F.Cu at (92.0, 49.3)
- added REF**: VIA-0.6mm, WiRoc:VIA-0.6mm, F.Cu at (79.4, 82.8)
- added REF**: VIA-0.6mm, WiRoc:VIA-0.6mm, F.Cu at (79.4, 81.1)
- added REF**: VIA-0.6mm, WiRoc:VIA-0.6mm, F.Cu at (69.4, 91.8)
- added REF**: VIA-0.6mm, WiRoc:VIA-0.6mm, F.Cu at (52.3, 56.0)
- added REF**: VIA-0.6mm, WiRoc:VIA-0.6mm, F.Cu at (72.6, 81.7)
- added REF**: VIA-0.6mm, WiRoc:VIA-0.6mm, F.Cu at (61.9, 76.6)
- added REF**: VIA-0.6mm, WiRoc:VIA-0.6mm, F.Cu at (71.2, 81.7)
- added REF**: VIA-0.6mm, WiRoc:VIA-0.6mm, F.Cu at (49.8, 52.4)
- added REF**: VIA-0.6mm, WiRoc:VIA-0.6mm, F.Cu at (59.3, 72.5)
- added REF**: VIA-0.6mm, WiRoc:VIA-0.6mm, F.Cu at (62.8, 70.1)
- added REF**: VIA-0.6mm, WiRoc:VIA-0.6mm, F.Cu at (62.8, 68.2)
- added REF**: VIA-0.6mm, WiRoc:VIA-0.6mm, F.Cu at (62.7, 66.2)
- added REF**: VIA-0.6mm, WiRoc:VIA-0.6mm, F.Cu at (59.4, 63.5)
- added REF**: VIA-0.6mm, WiRoc:VIA-0.6mm, F.Cu at (76.8, 84.0)
- added REF**: VIA-0.6mm, WiRoc:VIA-0.6mm, F.Cu at (70.4, 77.7)
- added REF**: VIA-0.6mm, WiRoc:VIA-0.6mm, F.Cu at (74.9, 104.1)
- added REF**: VIA-0.6mm, WiRoc:VIA-0.6mm, F.Cu at (89.7, 84.5)
- added REF**: VIA-0.6mm, WiRoc:VIA-0.6mm, F.Cu at (92.4, 94.9)
- added REF**: VIA-0.6mm, WiRoc:VIA-0.6mm, F.Cu at (92.3, 92.3)
- added REF**: VIA-0.6mm, WiRoc:VIA-0.6mm, F.Cu at (93.8, 107.6)
- added REF**: VIA-0.6mm, WiRoc:VIA-0.6mm, F.Cu at (92.2, 104.9)
- added REF**: VIA-0.6mm, WiRoc:VIA-0.6mm, F.Cu at (77.4, 92.1)
- added REF**: VIA-0.6mm, WiRoc:VIA-0.6mm, F.Cu at (79.5, 90.5)
- added REF**: VIA-0.6mm, WiRoc:VIA-0.6mm, F.Cu at (69.0, 79.3)
- added REF**: VIA-0.6mm, WiRoc:VIA-0.6mm, F.Cu at (68.4, 80.2)
- added REF**: VIA-0.6mm, WiRoc:VIA-0.6mm, F.Cu at (65.2, 80.4)
- added REF**: VIA-0.6mm, WiRoc:VIA-0.6mm, F.Cu at (75.2, 83.9)
- added REF**: VIA-0.6mm, WiRoc:VIA-0.6mm, F.Cu at (63.6, 82.0)
- added REF**: VIA-0.6mm, WiRoc:VIA-0.6mm, F.Cu at (67.0, 81.9)
- added REF**: VIA-0.6mm, WiRoc:VIA-0.6mm, F.Cu at (58.8, 87.5)
- added REF**: VIA-0.6mm, WiRoc:VIA-0.6mm, F.Cu at (58.7, 97.9)
- added REF**: VIA-0.6mm, WiRoc:VIA-0.6mm, F.Cu at (65.9, 102.8)
- added REF**: VIA-0.6mm, WiRoc:VIA-0.6mm, F.Cu at (60.9, 102.0)
- added REF**: VIA-0.6mm, WiRoc:VIA-0.6mm, F.Cu at (69.6, 96.0)
- added REF**: VIA-0.6mm, WiRoc:VIA-0.6mm, F.Cu at (69.6, 93.9)
- added REF**: VIA-0.6mm, WiRoc:VIA-0.6mm, F.Cu at (62.7, 86.3)
- added REF**: VIA-0.6mm, WiRoc:VIA-0.6mm, F.Cu at (62.7, 85.2)
- added REF**: VIA-0.6mm, WiRoc:VIA-0.6mm, F.Cu at (57.2, 110.5)
- added REF**: VIA-0.6mm, WiRoc:VIA-0.6mm, F.Cu at (62.7, 84.1)
- added REF**: VIA-0.6mm, WiRoc:VIA-0.6mm, F.Cu at (74.8, 98.6)
- added REF**: VIA-0.6mm, WiRoc:VIA-0.6mm, F.Cu at (76.9, 94.0)
- added REF**: VIA-0.6mm, WiRoc:VIA-0.6mm, F.Cu at (76.0, 92.6)
- added REF**: VIA-0.6mm, WiRoc:VIA-0.6mm, F.Cu at (92.8, 101.1)
- added REF**: VIA-0.6mm, WiRoc:VIA-0.6mm, F.Cu at (82.9, 89.7)
- added REF**: VIA-0.6mm, WiRoc:VIA-0.6mm, F.Cu at (85.6, 79.3)
- added REF**: VIA-0.6mm, WiRoc:VIA-0.6mm, F.Cu at (85.0, 81.8)
- added REF**: VIA-0.6mm, WiRoc:VIA-0.6mm, F.Cu at (94.2, 95.3)
- added REF**: VIA-0.6mm, WiRoc:VIA-0.6mm, F.Cu at (91.2, 108.8)
- added REF**: VIA-0.6mm, WiRoc:VIA-0.6mm, F.Cu at (62.7, 110.6)
- added REF**: VIA-0.6mm, WiRoc:VIA-0.6mm, F.Cu at (87.3, 87.1)
- added REF**: VIA-0.6mm, WiRoc:VIA-0.6mm, F.Cu at (87.5, 89.7)
- added REF**: VIA-0.6mm, WiRoc:VIA-0.6mm, F.Cu at (83.3, 79.5)
- added REF**: VIA-0.6mm, WiRoc:VIA-0.6mm, F.Cu at (53.5, 73.3)
- added REF**: VIA-0.6mm, WiRoc:VIA-0.6mm, F.Cu at (53.6, 63.4)
- added REF**: VIA-0.6mm, WiRoc:VIA-0.6mm, F.Cu at (76.8, 82.7)
- added REF**: VIA-0.6mm, WiRoc:VIA-0.6mm, F.Cu at (82.0, 84.1)
- added REF**: VIA-0.6mm, WiRoc:VIA-0.6mm, F.Cu at (82.0, 86.3)
- added REF**: VIA-0.6mm, WiRoc:VIA-0.6mm, F.Cu at (82.0, 88.3)
- added REF**: VIA-0.6mm, WiRoc:VIA-0.6mm, F.Cu at (79.1, 92.9)
- added REF**: VIA-0.6mm, WiRoc:VIA-0.6mm, F.Cu at (76.9, 95.6)
- added REF**: VIA-0.6mm, WiRoc:VIA-0.6mm, F.Cu at (66.9, 92.2)
- added REF**: VIA-0.6mm, WiRoc:VIA-0.6mm, F.Cu at (69.9, 82.0)
- added REF**: VIA-0.6mm, WiRoc:VIA-0.6mm, F.Cu at (61.9, 79.2)
- added REF**: VIA-0.6mm, WiRoc:VIA-0.6mm, F.Cu at (72.3, 78.9)
- added REF**: VIA-0.6mm, WiRoc:VIA-0.6mm, F.Cu at (51.1, 108.4)
- added REF**: VIA-0.6mm, WiRoc:VIA-0.6mm, F.Cu at (74.0, 79.9)
- added REF**: VIA-0.6mm, WiRoc:VIA-0.6mm, F.Cu at (73.9, 78.9)
- R4: value 1K -> 24K-1%
- moved TP10 43.2 mm to (83.3, 54.8), turned to 90 degrees
- moved TP1 25.4 mm to (84.2, 103.7)
- moved REF** 19.1 mm to (65.4, 97.2), turned to 90 degrees
- moved REF** 18.3 mm to (66.8, 97.2), turned to 90 degrees
- moved REF** 17.7 mm to (68.5, 97.2), turned to 90 degrees
- moved REF** 17.2 mm to (74.7, 96.6), turned to 90 degrees
- moved REF** 16.8 mm to (68.6, 98.6), turned to 90 degrees
- moved L1 14.7 mm to (66.8, 94.4), turned to 180 degrees
- moved R11 14.6 mm to (92.7, 67.5), turned to 180 degrees
- moved R1 14.2 mm to (74.6, 94.3), turned to 90 degrees
- moved R3 13.5 mm to (73.0, 94.3), turned to 90 degrees
- moved TP3 13.1 mm to (80.3, 85.2), turned to 90 degrees
- moved C1 13.1 mm to (79.7, 88.4), turned to 0 degrees
- moved C3 12.2 mm to (65.2, 82.8), turned to 90 degrees
- moved R2 12.1 mm to (79.5, 86.3), turned to 180 degrees
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Routing:
- net BAT: track 5.34 -> 49.3 mm, vias 2 -> 0
- net GND: track 34.4 -> 62.9 mm
- net N_VBUSEN: track 56.1 -> 28.2 mm, vias 2 -> 3
- net VDD_5V: track 121.0 -> 143.0 mm, vias 3 -> 4
- net LORAEN: track 32.0 -> 50.2 mm
- net UART1_TX: track 25.2 -> 41.0 mm
- net IRQ: track 56.0 -> 40.2 mm, vias 2 -> 0
- net VBUS: track 54.7 -> 69.8 mm, vias 2 -> 0
- net UART1_RX: track 29.8 -> 43.4 mm
- net SDA: track 98.6 -> 85.3 mm, vias 2 -> 0
- net SCK: track 100.6 -> 87.9 mm
- net Net-(D1-Pad2): track 17.2 -> 30.0 mm
- net PWRON: track 36.9 -> 49.0 mm, vias 3 -> 4
- net EXTEN: track 52.2 -> 63.9 mm
- net Net-(R13-Pad2): track 15.5 -> 27.2 mm
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- removed copper zone on B.Cu, net BAT
Other:
- board text removed: "Rx"
- board text removed: "Tx"
