File: KiCad5/Hardware_NanoPi_v4/WiRoc_NanoPi_v1.sch (KiCad schematic (older format))
At the start: 57 parts, among them J1 Conn_01x02, J2 USB_Power_02x02, J3 Serial, J4 USB_Host_Data_02x02, J6 HAT_Conn_DBG, J7 NanoPIAir, J8 USB_Host_Data_02x02, J9 Conn_Coaxial, SW1 SW_SPST, U1 DRF1268DS, U2 OLED, U3 AXP209, U4 LP6226_SY7208, U5 SY6280, U6 BatteryPadM, U7 BatteryPadP

Commit message: etc
Parts:
- removed D4, D5: LED, Diode_SMD:D_0603_1608Metric, symbol WiRoc_NanoPi_v1-rescue:LED
- added C16: 1uF, Capacitor_SMD:C_0603_1608Metric, symbol WiRoc_NanoPi_v1-rescue:C
- added C17: 47uF, Capacitor_SMD:C_1210_3225Metric, symbol Device:C
- added C18: 4.7uF, Capacitor_SMD:C_0603_1608Metric, symbol WiRoc_NanoPi_v1-rescue:C
- added D1: LED_DUAL_ACCA, WiRoc:LED_Dual_1.7_1.6, symbol WiRoc:LED_DUAL_ACCA
- added R6: 1K, Resistor_SMD:R_0603_1608Metric, symbol WiRoc_NanoPi_v1-rescue:R
- C1, C10, C11, C3, C8: Manufacturer Guangdong Fenghua Advanced Tech -> Samsung Electro-Mechanics; ManufacturerPartNumber 0603B475K160NT -> CL10A475KO8NNNC
- C2, C6, C9: Manufacturer Guangdong Fenghua Advanced Tech -> Samsung Electro-Mechanics; ManufacturerPartNumber 0603X105K500NT -> CL10A105KB8NNNC
- C7: Manufacturer Guangdong Fenghua Advanced Tech -> Samsung Electro-Mechanics; ManufacturerPartNumber 0603CG101J500NT -> CL10C101JB8NNNC
- D3: Manufacturer Diodes Incorporated -> Changjiang Electronics Tech (CJ); ManufacturerPartNumber 1N5819HW-7-F -> B5817W
- J1: footprint Pin_Headers:Pin_Header_Straight_1x02_Pitch2.54mm -> WiRoc:Pin_Header_Straight_1x02_Pitch2.54mm
- J6: footprint Pin_Headers:Pin_Header_Straight_1x03_Pitch2.54mm -> WiRoc:Pin_Header_Straight_1x03_Pitch2.54mm
- R11, R12: Manufacturer Huaxin S&T -> Uniroyal Elec; ManufacturerPartNumber WR06X103JTL -> 0603WAF1002T5E
- R13, R14: LCSCPartNumber C21190 -> C25585; Manufacturer RALEC -> Uniroyal Elec; ManufacturerPartNumber RTT031001FTP -> 0603WAJ0102T5E
- R4: value 1K -> 24K-1%; Description 1KΩ (1001) ±1% -> (none); LCSCPartNumber C21190 -> C23352; Manufacturer RALEC -> Uniroyal Elec; ManufacturerPartNumber RTT031001FTP -> 0603WAF2402T5E
- R5: Manufacturer RALEC -> Uniroyal Elec; ManufacturerPartNumber RTT05R030FTP -> 0805W4F300MT5E
- R9: Manufacturer LIZ Elec -> Uniroyal Elec; ManufacturerPartNumber CR0603FA3601G -> 0603WAF3601T5E
- SW1: footprint Connector_PinHeader_2.54mm:PinHeader_1x02_P2.54mm_Vertical -> WiRoc:Pin_Header_Straight_1x02_Pitch2.54mm
- U4: Manufacturer lowpowersemi -> Silergy Corp; ManufacturerPartNumber LP6226B6F -> SY7208ABC
- U5: Manufacturer SILERGY -> Silergy Corp
Connections:
- net GND: now also C16.2, C17.1, C18.2
- net VDD_5V: now also C16.1, C17.2, C18.1
- net at U1.4 (L1): now also D1.2 (K1)
- net at U1.5 (L2): now also D1.3 (K2)
- net at R13.2, R14.2, U1.8 (VCC): now also R6.2
- net at R14.1: now also D1.1 (A1), R6.1
- net at R13.1: now also D1.4 (A2)
Other:
- moved on the sheet: R13, R14
