File: KiCad7/TestBoost/TestBoost.kicad_sch (KiCad schematic)
At the start: 11 parts, among them J1 Conn_01x02_Male, J2 USB_A, J3 Conn_01x02_Male, J4 Conn_01x03_Male

Commit message: diverse SRR etc
Parts:
- R2: LCSC Part # C270943 -> C321721
Changed lines of the file:
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@@
       (effects (font (size 1.27 1.27)) hide)
     )
-    (property "LCSC Part #" "C270943" (at 123.19 72.39 0)
+    (property "LCSC Part #" "C321721" (at 123.19 72.39 0)
       (effects (font (size 1.27 1.27)) hide)
     )
