File: KiCad7/Hardware_NanoPi_v7/RTC.kicad_sch (KiCad schematic)
At the start: 8 parts, among them U4 74LS73, U9 PCF8563T, Y1 32.768kHz

Commit message: merge after probably pushed from old laptop
Parts:
- U4, U9: JLCPCB Rotation Offset -90 -> 0
Changed lines of the file:
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@@
       (effects (font (size 1.27 1.27)) hide)
     )
-    (property "JLCPCB Rotation Offset" "-90" (at 180.34 38.1 0)
+    (property "JLCPCB Rotation Offset" "0" (at 180.34 38.1 0)
       (effects (font (size 1.27 1.27)) hide)
     )
@@
   (symbol (lib_id "power:GND") (at 101.6 80.01 0) (unit 1)
     (in_bom yes) (on_board yes) (dnp no)
-    (property "Reference" "#PWR024" (at 101.6 86.36 0)
+    (property "Reference" "#PWR01" (at 101.6 86.36 0)
       (effects (font (size 1.27 1.27)) hide)
     )
@@
     (instances
       (project "WiRoc_NanoPi"
-        (path "/8ba0b499-eaca-4cd5-a002-c6bdb610cc8c/34a3fa8a-641a-40bf-8a99-689cdb159b8f"
-          (reference "#PWR024") (unit 1)
-        )
         (path "/8ba0b499-eaca-4cd5-a002-c6bdb610cc8c/420ce888-9e08-49fd-b3f8-96e9de814cbc"
           (reference "#PWR01") (unit 1)
@@
       (effects (font (size 1.27 1.27)) hide)
     )
-    (property "JLCPCB Rotation Offset" "-90" (at 171.45 68.58 0)
+    (property "JLCPCB Rotation Offset" "0" (at 171.45 68.58 0)
       (effects (font (size 1.27 1.27)) hide)
     )
@@
   (symbol (lib_id "power:GND") (at 124.46 80.01 0) (unit 1)
     (in_bom yes) (on_board yes) (dnp no)
-    (property "Reference" "#PWR024" (at 124.46 86.36 0)
+    (property "Reference" "#PWR02" (at 124.46 86.36 0)
       (effects (font (size 1.27 1.27)) hide)
     )
@@
     (instances
       (project "WiRoc_NanoPi"
-        (path "/8ba0b499-eaca-4cd5-a002-c6bdb610cc8c/34a3fa8a-641a-40bf-8a99-689cdb159b8f"
-          (reference "#PWR024") (unit 1)
-        )
         (path "/8ba0b499-eaca-4cd5-a002-c6bdb610cc8c/420ce888-9e08-49fd-b3f8-96e9de814cbc"
           (reference "#PWR02") (unit 1)
@@
   (symbol (lib_id "power:GND") (at 180.34 48.26 0) (unit 1)
     (in_bom yes) (on_board yes) (dnp no)
-    (property "Reference" "#PWR024" (at 180.34 54.61 0)
+    (property "Reference" "#PWR037" (at 180.34 54.61 0)
       (effects (font (size 1.27 1.27)) hide)
     )
@@
     (instances
       (project "WiRoc_NanoPi"
-        (path "/8ba0b499-eaca-4cd5-a002-c6bdb610cc8c/34a3fa8a-641a-40bf-8a99-689cdb159b8f"
-          (reference "#PWR024") (unit 1)
-        )
         (path "/8ba0b499-eaca-4cd5-a002-c6bdb610cc8c/420ce888-9e08-49fd-b3f8-96e9de814cbc"
           (reference "#PWR037") (unit 1)
@@
       (effects (font (size 1.27 1.27)) hide)
     )
-    (property "JLCPCB Rotation Offset" "-90" (at 124.46 63.5 0)
+    (property "JLCPCB Rotation Offset" "0" (at 124.46 63.5 0)
       (effects (font (size 1.27 1.27)) hide)
     )
@@
       (effects (font (size 1.27 1.27)) hide)
     )
-    (property "JLCPCB Rotation Offset" "-90" (at 161.29 39.37 0)
+    (property "JLCPCB Rotation Offset" "0" (at 161.29 39.37 0)
       (effects (font (size 1.27 1.27)) hide)
     )
@@
   (symbol (lib_id "power:GND") (at 90.17 80.01 0) (unit 1)
     (in_bom yes) (on_board yes) (dnp no)
-    (property "Reference" "#PWR024" (at 90.17 86.36 0)
+    (property "Reference" "#PWR03" (at 90.17 86.36 0)
       (effects (font (size 1.27 1.27)) hide)
     )
@@
     (instances
       (project "WiRoc_NanoPi"
-        (path "/8ba0b499-eaca-4cd5-a002-c6bdb610cc8c/34a3fa8a-641a-40bf-8a99-689cdb159b8f"
-          (reference "#PWR024") (unit 1)
-        )
         (path "/8ba0b499-eaca-4cd5-a002-c6bdb610cc8c/420ce888-9e08-49fd-b3f8-96e9de814cbc"
           (reference "#PWR03") (unit 1)
@@
   (symbol (lib_id "power:GND") (at 181.61 91.44 0) (unit 1)
     (in_bom yes) (on_board yes) (dnp no)
-    (property "Reference" "#PWR024" (at 181.61 97.79 0)
+    (property "Reference" "#PWR022" (at 181.61 97.79 0)
       (effects (font (size 1.27 1.27)) hide)
     )
@@
     (instances
       (project "WiRoc_NanoPi"
-        (path "/8ba0b499-eaca-4cd5-a002-c6bdb610cc8c/34a3fa8a-641a-40bf-8a99-689cdb159b8f"
-          (reference "#PWR024") (unit 1)
-        )
         (path "/8ba0b499-eaca-4cd5-a002-c6bdb610cc8c/420ce888-9e08-49fd-b3f8-96e9de814cbc"
           (reference "#PWR022") (unit 1)
