File: KiCad7/Hardware_NanoPi_v7/Serial.kicad_sch (KiCad schematic)
At the start: 7 parts, among them J4 Conn_01x03_Socket, U8 SP3232ECY-L

Commit message: merge after probably pushed from old laptop
Parts:
- C20, C21, C22, C23, C24: ThroughHole (none) -> FALSE
- J4: value Conn_01x03_Socket -> Conn_01x09_Socket; footprint Connector_PinSocket_1.27mm:PinSocket_1x03_P1.27mm_Vertical -> Connector_PinSocket_1.27mm:PinSocket_1x09_P1.27mm_Vertical; symbol Connector:Conn_01x03_Socket -> Connector:Conn_01x09_Socket; ThroughHole (none) -> TRUE
- U8: JLCPCB Rotation Offset -90 -> 0; LCSC Part # C31142 -> C3028967
Connections:
- net GND: now also J4.3 (Pin_3), J4.8 (Pin_8); no longer J4.1 (Pin_1)
- net at U8.7 (T2OUT): now also J4.1 (Pin_1); no longer J4.3 (Pin_3)
- new net ToPWRBTN: J4.9 (Pin_9)
- no-connect marks 4 -> 8
Changed lines of the file:
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@@
   (junction (at 77.47 49.53) (diameter 0) (color 0 0 0 0)
   )
+  (no_connect (at 135.89 97.79))
   (no_connect (at 57.15 82.55))
+  (no_connect (at 97.79 82.55))
   (no_connect (at 97.79 92.71))
-  (no_connect (at 97.79 82.55))
+  (no_connect (at 135.89 90.17))
+  (no_connect (at 135.89 92.71))
   (no_connect (at 57.15 92.71))
-  (wire (pts (xy 97.79 87.63) (xy 135.89 87.63))
+  (no_connect (at 135.89 95.25))
+  (wire (pts (xy 104.14 87.63) (xy 97.79 87.63))
     (stroke (width 0) (type default))
   )
@@
     (stroke (width 0) (type default))
   )
+  (wire (pts (xy 104.14 82.55) (xy 135.89 82.55))
+    (stroke (width 0) (type default))
+  )
   (wire (pts (xy 97.79 64.77) (xy 104.14 64.77))
+    (stroke (width 0) (type default))
+  )
+  (wire (pts (xy 104.14 82.55) (xy 104.14 87.63))
     (stroke (width 0) (type default))
   )
@@
     )
   )
+  (global_label "ToPWRBTN" (shape input) (at 135.89 102.87 180) (fields_autoplaced)
+    (effects (font (size 1.524 1.524)) (justify right))
+    (property "Intersheetrefs" "${INTERSHEET_REFS}" (at 121.4818 102.87 0)
+      (effects (font (size 1.27 1.27)) (justify right) hide)
+    )
+  )
   (global_label "UART2_RX" (shape output) (at 57.15 97.79 180) (fields_autoplaced)
     (effects (font (size 1.524 1.524)) (justify right))
@@
       (effects (font (size 1.27 1.27)) hide)
     )
+    (property "ThroughHole" "FALSE" (at 104.14 77.47 0)
+      (effects (font (size 1.27 1.27)) hide)
+    )
     (pin "1")
     (pin "2")
@@
       (effects (font (size 1.27 1.27)) hide)
     )
+    (property "ThroughHole" "FALSE" (at 52.07 60.96 0)
+      (effects (font (size 1.27 1.27)) hide)
+    )
     (pin "1")
     (pin "2")
@@
     )
     (property "JLCPCB Rotation Offset" "" (at 104.14 69.85 0)
+      (effects (font (size 1.27 1.27)) hide)
+    )
+    (property "ThroughHole" "FALSE" (at 104.14 69.85 0)
       (effects (font (size 1.27 1.27)) hide)
     )
@@
       (effects (font (size 1.27 1.27)) hide)
     )
-    (property "LCSC Part #" "C31142" (at 77.47 80.01 0)
-      (effects (font (size 1.27 1.27)) hide)
-    )
-    (property "JLCPCB Rotation Offset" "-90" (at 77.47 80.01 0)
+    (property "LCSC Part #" "C3028967" (at 77.47 80.01 0)
+      (effects (font (size 1.27 1.27)) hide)
+    )
+    (property "JLCPCB Rotation Offset" "0" (at 77.47 80.01 0)
       (effects (font (size 1.27 1.27)) hide)
     )
@@
     (instances
       (project "WiRoc_NanoPi"
-        (path "/8ba0b499-eaca-4cd5-a002-c6bdb610cc8c"
+        (path "/8ba0b499-eaca-4cd5-a002-c6bdb610cc8c/34a3fa8a-641a-40bf-8a99-689cdb159b8f"
           (reference "U8") (unit 1)
         )
-        (path "/8ba0b499-eaca-4cd5-a002-c6bdb610cc8c/34a3fa8a-641a-40bf-8a99-689cdb159b8f"
-          (reference "U8") (unit 1)
-        )
       )
     )
@@
       (effects (font (size 1.27 1.27)) hide)
     )
+    (property "ThroughHole" "FALSE" (at 104.14 60.96 0)
+      (effects (font (size 1.27 1.27)) hide)
+    )
     (pin "1")
     (pin "2")
@@
     )
   )
-  (symbol (lib_id "Connector:Conn_01x03_Socket") (at 140.97 85.09 0) (unit 1)
+  (symbol (lib_id "Connector:Conn_01x09_Socket") (at 140.97 92.71 0) (unit 1)
     (in_bom no) (on_board yes) (dnp no) (fields_autoplaced)
-    (property "Reference" "J4" (at 142.24 83.82 0)
-      (effects (font (size 1.27 1.27)) (justify left))
-    )
-    (property "Value" "Conn_01x03_Socket" (at 142.24 86.36 0)
-      (effects (font (size 1.27 1.27)) (justify left))
-    )
-    (property "Footprint" "Connector_PinSocket_1.27mm:PinSocket_1x03_P1.27mm_Vertical" (at 140.97 85.09 0)
-      (effects (font (size 1.27 1.27)) hide)
-    )
-    (property "Datasheet" "~" (at 140.97 85.09 0)
-      (effects (font (size 1.27 1.27)) hide)
-    )
-    (property "IncludeInBOM" "FALSE" (at 140.97 85.09 0)
+    (property "Reference" "J4" (at 142.24 91.44 0)
+      (effects (font (size 1.27 1.27)) (justify left))
+    )
+    (property "Value" "Conn_01x09_Socket" (at 142.24 93.98 0)
+      (effects (font (size 1.27 1.27)) (justify left))
+    )
+    (property "Footprint" "Connector_PinSocket_1.27mm:PinSocket_1x09_P1.27mm_Vertical" (at 140.97 92.71 0)
+      (effects (font (size 1.27 1.27)) hide)
+    )
+    (property "Datasheet" "~" (at 140.97 92.71 0)
+      (effects (font (size 1.27 1.27)) hide)
+    )
+    (property "IncludeInBOM" "FALSE" (at 140.97 92.71 0)
+      (effects (font (size 1.27 1.27)) hide)
+    )
+    (property "ThroughHole" "TRUE" (at 140.97 92.71 0)
       (effects (font (size 1.27 1.27)) hide)
     )
@@
     (pin "2")
     (pin "3")
+    (pin "8")
+    (pin "7")
+    (pin "5")
+    (pin "4")
+    (pin "6")
+    (pin "9")
     (instances
       (project "WiRoc_NanoPi"
@@
       (effects (font (size 1.27 1.27)) hide)
     )
+    (property "ThroughHole" "FALSE" (at 87.63 49.53 0)
+      (effects (font (size 1.27 1.27)) hide)
+    )
     (pin "1")
     (pin "2")
@@
     )
   )
-  (symbol (lib_id "power:GND") (at 135.89 82.55 270) (unit 1)
-    (in_bom yes) (on_board yes) (dnp no)
-    (property "Reference" "#PWR0115" (at 129.54 82.55 0)
-      (effects (font (size 1.27 1.27)) hide)
-    )
-    (property "Value" "GND" (at 132.08 82.55 0)
-      (effects (font (size 1.27 1.27)))
-    )
-    (property "Footprint" "" (at 135.89 82.55 0)
-      (effects (font (size 1.27 1.27)) hide)
-    )
-    (property "Datasheet" "" (at 135.89 82.55 0)
-      (effects (font (size 1.27 1.27)) hide)
-    )
-    (pin "1")
-    (instances
-      (project "WiRoc_NanoPi"
-        (path "/8ba0b499-eaca-4cd5-a002-c6bdb610cc8c"
-          (reference "#PWR0115") (unit 1)
-        )
+  (symbol (lib_id "power:GND") (at 135.89 87.63 270) (unit 1)
+    (in_bom yes) (on_board yes) (dnp no)
+    (property "Reference" "#PWR031" (at 129.54 87.63 0)
+      (effects (font (size 1.27 1.27)) hide)
+    )
+    (property "Value" "GND" (at 132.08 87.63 0)
+      (effects (font (size 1.27 1.27)))
+    )
+    (property "Footprint" "" (at 135.89 87.63 0)
+      (effects (font (size 1.27 1.27)) hide)
+    )
+    (property "Datasheet" "" (at 135.89 87.63 0)
+      (effects (font (size 1.27 1.27)) hide)
+    )
+    (pin "1")
+    (instances
+      (project "WiRoc_NanoPi"
         (path "/8ba0b499-eaca-4cd5-a002-c6bdb610cc8c/34a3fa8a-641a-40bf-8a99-689cdb159b8f"
           (reference "#PWR031") (unit 1)
         )
       )
+    )
+  )
+  (symbol (lib_id "power:GND") (at 135.89 100.33 270) (unit 1)
+    (in_bom yes) (on_board yes) (dnp no)
+    (property "Reference" "#PWR014" (at 129.54 100.33 0)
+      (effects (font (size 1.27 1.27)) hide)
+    )
+    (property "Value" "GND" (at 132.6388 100.457 90)
+      (effects (font (size 1.27 1.27)) (justify right))
+    )
+    (property "Footprint" "" (at 135.89 100.33 0)
+      (effects (font (size 1.27 1.27)) hide)
+    )
+    (property "Datasheet" "" (at 135.89 100.33 0)
+      (effects (font (size 1.27 1.27)) hide)
+    )
+    (pin "1")
+    (instances
+      (project "WiRoc_NanoPi"
+        (path "/8ba0b499-eaca-4cd5-a002-c6bdb610cc8c/34a3fa8a-641a-40bf-8a99-689cdb159b8f"
+          (reference "#PWR014") (unit 1)
+        )
+      )
