File: KiCad7/Hardware_NanoPi_v7/WiRoc_NanoPi.kicad_pcb (KiCad board)
At the start: 4 copper layers, 48 x 68.7 mm, 75 parts, among them J1 Conn_01x02_Socket, J10 Conn_01x06_Socket, J11 Conn_01x04_Socket, J12 Conn_01x02_Socket, J2 Conn_01x04, J3 Conn_01x02_Socket, J4 Conn_01x03_Socket, J5 Conn_01x05_Socket, J6 HAT_Conn_DBG, J7 NanoPIAir, J8 Conn_01x06, J9 Conn_Coaxial, SW1 SW_SPST, U1 DRF1268DS, U2 OLED, U3 AXP209, U4 74LS73, U5 SY6280, U6 BatteryPadM, U7 BatteryPadP, U8 SP3232ECY-L, U9 PCF8563T, Y1 32.768kHz

Commit message: merge after probably pushed from old laptop
Parts:
- removed J11: Conn_01x04_Socket, Connector_PinSocket_1.27mm:PinSocket_1x04_P1.27mm_Vertical
- removed J12, J3: Conn_01x02_Socket, Connector_PinSocket_1.27mm:PinSocket_1x02_P1.27mm_Vertical
- J1: value Conn_01x02_Socket -> Conn_02x05_Odd_Even; footprint Connector_PinSocket_1.27mm:PinSocket_1x02_P1.27mm_Vertical -> Connector_PinHeader_1.27mm:PinHeader_2x05_P1.27mm_Vertical; moved to F.Cu
- J10: value Conn_01x06_Socket -> Conn_01x09_Socket; footprint Connector_PinSocket_1.27mm:PinSocket_1x06_P1.27mm_Vertical -> Connector_PinSocket_1.27mm:PinSocket_1x09_P1.27mm_Vertical
- J4: value Conn_01x03_Socket -> Conn_01x09_Socket; footprint Connector_PinSocket_1.27mm:PinSocket_1x03_P1.27mm_Vertical -> Connector_PinSocket_1.27mm:PinSocket_1x09_P1.27mm_Vertical
- J5: value Conn_01x05_Socket -> Conn_01x04_Socket; footprint Connector_PinSocket_1.27mm:PinSocket_1x05_P1.27mm_Vertical -> Connector_PinSocket_1.27mm:PinSocket_1x04_P1.27mm_Vertical
- moved J1 14.6 mm to (49.2, 62.5), turned to 90 degrees
- moved J10 3.81 mm to (51.0, 77.0)
- moved J4 2.54 mm to (51.0, 94.8), turned to 180 degrees
- moved J5 1.27 mm to (51.0, 55.4)
- moved U2 0.50 mm to (88.2, 48.3)
Connections:
- J1 pad 1: GND -> SYS_3.3V
- J1 pad 2: VBUS -> Net-(J1-Pin_2)
- J10 pad 1: GND -> VBUS
- J10 pad 2: USBHost-DP1 -> GND
- J10 pad 3: USBHost-DM1 -> unconnected-(J10-Pin_3-Pad3)
- J10 pad 4: VDD_5V -> GND
- J10 pad 5: USBHost-DP2 -> USBHost-DP1
- J10 pad 6: USBHost-DM2 -> USBHost-DM1
- J2 pad 1: unconnected-(J2-Pin_1-Pad1) -> Net-(J1-Pin_4)
- J2 pad 2: unconnected-(J2-Pin_2-Pad2) -> Net-(J1-Pin_7)
- J2 pad 3: unconnected-(J2-Pin_3-Pad3) -> Net-(J1-Pin_9)
- J4 pad 1: GND -> Net-(J4-Pin_1)
- J4 pad 3: Net-(J4-Pin_3) -> GND
- J8 pad 4: unconnected-(J8-Pin_4-Pad4) -> Net-(J1-Pin_2)
- R4 pad 1: Net-(J3-Pin_2) -> ToPWRBTN
- U8 pad 7: Net-(J4-Pin_3) -> Net-(J4-Pin_1)
Routing:
- net Net-(J1-Pin_2): track 0.00 -> 34.0 mm
- net SRR_NRST: track 75.9 -> 105.6 mm
- net SYS_3.3V: track 123.9 -> 149.1 mm
- net Net-(J1-Pin_7): track 0.00 -> 19.2 mm, vias 0 -> 1
- net Net-(J1-Pin_4): track 0.00 -> 18.2 mm
- net Net-(J1-Pin_9): track 0.00 -> 17.5 mm, vias 0 -> 1
- net Net-(J4-Pin_3): track 14.9 -> 0.00 mm
- net Net-(J4-Pin_1): track 0.00 -> 14.9 mm
- net ToPWRBTN: track 0.00 -> 5.66 mm
- net Net-(J3-Pin_2): track 5.66 -> 0.00 mm
- net VBUS: track 31.1 -> 31.7 mm
- net SCK: track 103.4 -> 102.9 mm
Other:
- board text added: "Rx Tx Gnd"
- board text removed: "Gnd Tx Rx"
