File: KiCad7/Hardware_NanoPi_v7/WiRoc_NanoPi.kicad_sch (KiCad schematic)
At the start: 60 parts, among them J1 Conn_01x02_Socket, J10 Conn_01x06_Socket, J11 Conn_01x04_Socket, J12 Conn_01x02_Socket, J2 Conn_01x04, J3 Conn_01x02_Socket, J5 Conn_01x05_Socket, J6 HAT_Conn_DBG, J7 NanoPIAir, J8 Conn_01x06, J9 Conn_Coaxial, SW1 SW_SPST, U1 DRF1268DS, U2 OLED, U3 AXP209, U5 SY6280, U6 BatteryPadM, U7 BatteryPadP

Commit message: merge after probably pushed from old laptop
Parts:
- removed J1, J12, J3: Conn_01x02_Socket, Connector_PinSocket_1.27mm:PinSocket_1x02_P1.27mm_Vertical, symbol Connector:Conn_01x02_Socket
- removed J11: Conn_01x04_Socket, Connector_PinSocket_1.27mm:PinSocket_1x04_P1.27mm_Vertical, symbol Connector:Conn_01x04_Socket
- added J1: Conn_02x05_Odd_Even, Connector_PinHeader_1.27mm:PinHeader_2x05_P1.27mm_Vertical, symbol Connector_Generic:Conn_02x05_Odd_Even
- C26, C27, L3, R15, R16: ThroughHole (none) -> FALSE
- J10: value Conn_01x06_Socket -> Conn_01x09_Socket; footprint Connector_PinSocket_1.27mm:PinSocket_1x06_P1.27mm_Vertical -> Connector_PinSocket_1.27mm:PinSocket_1x09_P1.27mm_Vertical; symbol Connector:Conn_01x06_Socket -> Connector:Conn_01x09_Socket
- J2: ThroughHole (none) -> TRUE
- J5: value Conn_01x05_Socket -> Conn_01x04_Socket; footprint Connector_PinSocket_1.27mm:PinSocket_1x05_P1.27mm_Vertical -> Connector_PinSocket_1.27mm:PinSocket_1x04_P1.27mm_Vertical; symbol Connector:Conn_01x05_Socket -> Connector:Conn_01x04_Socket
- U10: JLCPCB Rotation Offset 180 -> 0
- U5: JLCPCB Rotation Offset -90 -> 90
Connections:
- net GND: now also J10.2 (Pin_2), J10.4 (Pin_4), J1.3 (Pin_3), J1.5 (Pin_5); no longer J10.1 (Pin_1)
- net SRR_NRST: now also J1.10 (Pin_10)
- net SYS_3.3V: now also J1.1 (Pin_1)
- net USBHost-DM1: now also J10.6 (Pin_6); no longer J10.3 (Pin_3)
- net USBHost-DM2: now also J10.9 (Pin_9); no longer J10.6 (Pin_6)
- net USBHost-DP1: now also J10.5 (Pin_5); no longer J10.2 (Pin_2)
- net USBHost-DP2: now also J10.8 (Pin_8); no longer J10.5 (Pin_5)
- net VBUS: now also J10.1 (Pin_1)
- net VDD_5V: now also J10.7 (Pin_7); no longer J10.4 (Pin_4)
- net ToPWRBTN: now reaches R4.1
- net at J2.1 (Pin_1): now also J1.4 (Pin_4)
- net at J2.2 (Pin_2): now also J1.7 (Pin_7)
- net at J2.3 (Pin_3): now also J1.9 (Pin_9)
- net at J8.4 (Pin_4): now also J1.2 (Pin_2)
- no-connect marks 57 -> 50
Other:
- moved on the sheet: J2, J8
