File: KiCad7/Hardware_NanoPi_v7_ConnectorPlate/Hardware_NanoPi_v7_ConnectorPlate.kicad_pcb (KiCad board)
At the start: 2 copper layers, 16 x 57.5 mm, 11 parts, among them J10 Conn_01x02, J11 Conn_01x02, J12 Conn_01x02, J2 USB_Host_Data_02x02, J3 USB_Host_Data_02x02, J4 USB_Power_02x02, J5 Conn_01x03, J6 Conn_01x02, J7 Conn_01x06, J8 Conn_01x03, J9 Conn_01x02

Commit message: merge after probably pushed from old laptop
Parts:
- removed J7: Conn_01x06, Connector_PinHeader_1.27mm:PinHeader_1x06_P1.27mm_Horizontal
- removed J9: Conn_01x02, Connector_PinHeader_1.27mm:PinHeader_1x02_P1.27mm_Horizontal
- added U1: USBLC6-2P6, Package_TO_SOT_SMD:SOT-666, F.Cu at (110.2, 84.2)
- added U2: USBLC6-2P6, Package_TO_SOT_SMD:SOT-666, F.Cu at (110.3, 79.5)
- added U3: USBLC6-2P6, Package_TO_SOT_SMD:SOT-666, F.Cu at (110.5, 58.0)
- J10: value Conn_01x02 -> Conn_01x04; footprint Connector_PinHeader_1.27mm:PinHeader_1x02_P1.27mm_Horizontal -> Connector_PinHeader_1.27mm:PinHeader_1x04_P1.27mm_Horizontal
- J6: value Conn_01x02 -> Conn_01x09; footprint Connector_PinHeader_1.27mm:PinHeader_1x02_P1.27mm_Horizontal -> Connector_PinHeader_1.27mm:PinHeader_1x09_P1.27mm_Horizontal
- J8: value Conn_01x03 -> Conn_01x09; footprint Connector_PinHeader_1.27mm:PinHeader_1x03_P1.27mm_Horizontal -> Connector_PinHeader_1.27mm:PinHeader_1x09_P1.27mm_Horizontal
- moved J6 1.27 mm to (114.0, 74.3)
- moved J11 0.11 mm to (106.0, 93.8)
Connections:
- J2 pad 2: USBHost-DM1 -> Net-(J2-Pin_2)
- J2 pad 3: USBHost-DP1 -> Net-(J2-Pin_3)
- J3 pad 2: USBHost-DM2 -> Net-(J3-Pin_2)
- J3 pad 3: USBHost-DP2 -> Net-(J3-Pin_3)
Routing:
- net Net-(J3-Pin_2): track 0.00 -> 11.3 mm
- net Net-(J2-Pin_3): track 0.00 -> 7.81 mm
- net GND: track 0.00 -> 7.65 mm, vias 0 -> 16
- net VDD_5V: track 29.6 -> 37.0 mm
- net VBUS: track 26.2 -> 31.5 mm
- net Net-(J3-Pin_3): track 0.00 -> 5.01 mm
- net USBHost-DP1: track 7.84 -> 4.51 mm, vias 0 -> 1
- net Net-(J2-Pin_2): track 0.00 -> 3.30 mm
- net USBHost-DM1: track 6.60 -> 4.05 mm
- net USBHost-DP2: track 6.16 -> 3.76 mm
- net USBHost-DM2: track 6.74 -> 4.51 mm, vias 0 -> 1
- net R2IN: track 14.7 -> 16.9 mm
- net PWRBTN: track 48.5 -> 49.8 mm
Other:
- board size 16 x 57.5 mm -> 16 x 60 mm
