File: KiCad7/Hardware_NanoPi_v7_ConnectorPlate/Hardware_NanoPi_v7_ConnectorPlate.kicad_sch (KiCad schematic)
At the start: 11 parts, among them J10 Conn_01x02, J11 Conn_01x02, J12 Conn_01x02, J2 USB_Power_02x02, J4 USB_Host_Data_02x02, J5 Conn_01x03, J6 Conn_01x02, J7 Conn_01x06, J8 Conn_01x03, J8 USB_Host_Data_02x02, J9 Conn_01x02

Commit message: merge after probably pushed from old laptop
Parts:
- removed J7: Conn_01x06, Connector_PinHeader_1.27mm:PinHeader_1x06_P1.27mm_Horizontal, symbol Connector_Generic:Conn_01x06
- removed J9: Conn_01x02, Connector_PinHeader_1.27mm:PinHeader_1x02_P1.27mm_Horizontal, symbol Connector_Generic:Conn_01x02
- added U1, U2, U3: USBLC6-2P6, Package_TO_SOT_SMD:SOT-666, symbol Power_Protection:USBLC6-2P6
- J10: value Conn_01x02 -> Conn_01x04; footprint Connector_PinHeader_1.27mm:PinHeader_1x02_P1.27mm_Horizontal -> Connector_PinHeader_1.27mm:PinHeader_1x04_P1.27mm_Horizontal; symbol Connector_Generic:Conn_01x02 -> Connector_Generic:Conn_01x04
- J6: value Conn_01x02 -> Conn_01x09; footprint Connector_PinHeader_1.27mm:PinHeader_1x02_P1.27mm_Horizontal -> Connector_PinHeader_1.27mm:PinHeader_1x09_P1.27mm_Horizontal; symbol Connector_Generic:Conn_01x02 -> Connector_Generic:Conn_01x09
- J8: value Conn_01x03 -> Conn_01x09; footprint Connector_PinHeader_1.27mm:PinHeader_1x03_P1.27mm_Horizontal -> Connector_PinHeader_1.27mm:PinHeader_1x09_P1.27mm_Horizontal; symbol Connector_Generic:Conn_01x03 -> Connector_Generic:Conn_01x09
Connections:
- net GND: now also J6.4 (Pin_4), J8.8 (Pin_8), U1.2 (GND), U2.2 (GND), U3.2 (GND)
- net PWRBTN: now also J8.9 (Pin_9)
- net USBHost-DM1: now also J6.6 (Pin_6), U2.6 (I/O1); no longer J4.2 (Pin_2)
- net USBHost-DM2: now also J6.9 (Pin_9), U1.6 (I/O1); no longer J8.2 (Pin_2)
- net USBHost-DP1: now also J6.5 (Pin_5), U2.4 (I/O2); no longer J4.3 (Pin_3)
- net USBHost-DP2: now also J6.8 (Pin_8), U1.4 (I/O2); no longer J8.3 (Pin_3)
- net VBUS: now also U3.5 (VBUS)
- net VDD_5V: now also J6.7 (Pin_7), U1.5 (VBUS), U2.5 (VBUS)
- new net: J4.2 (Pin_2), U2.1 (I/O1)
- new net: J4.3 (Pin_3), U2.3 (I/O2)
- new net: J8.2 (Pin_2), U1.1 (I/O1)
- new net: J8.3 (Pin_3), U1.3 (I/O2)
- no-connect marks 4 -> 15
Other:
- moved on the sheet: J11, J12, J2, J4, J5, J8
