File: KiCad7/Hardware_WiRoc_v8/LED-Etc.kicad_sch (KiCad schematic)
At the start: 4 parts

Commit message: wiroc v8 layout work
Parts:
- R39, R40, R41: footprint Resistor_SMD:R_0603_1608Metric -> Resistor_SMD:R_0402_1005Metric
Changed lines of the file:
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@@
       (effects (font (size 1.27 1.27)))
     )
-    (property "Footprint" "Resistor_SMD:R_0603_1608Metric" (at 88.9 54.102 90)
+    (property "Footprint" "Resistor_SMD:R_0402_1005Metric" (at 88.9 54.102 90)
       (effects (font (size 1.27 1.27)) hide)
     )
@@
       (effects (font (size 1.27 1.27)))
     )
-    (property "Footprint" "Resistor_SMD:R_0603_1608Metric" (at 78.232 40.64 90)
+    (property "Footprint" "Resistor_SMD:R_0402_1005Metric" (at 78.232 40.64 90)
       (effects (font (size 1.27 1.27)) hide)
     )
@@
       (effects (font (size 1.27 1.27)))
     )
-    (property "Footprint" "Resistor_SMD:R_0603_1608Metric" (at 88.9 49.022 90)
+    (property "Footprint" "Resistor_SMD:R_0402_1005Metric" (at 88.9 49.022 90)
       (effects (font (size 1.27 1.27)) hide)
     )
