File: KiCad7/Hardware_WiRoc_v8/Processor.kicad_sch (KiCad schematic)
At the start: 21 parts

Commit message: wiroc v8 layout work
Parts:
- R19: footprint Resistor_SMD:R_0603_1608Metric -> Resistor_SMD:R_0402_1005Metric
Changed lines of the file:
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@@
       (effects (font (size 1.27 1.27)) (justify left))
     )
-    (property "Footprint" "Resistor_SMD:R_0603_1608Metric" (at 38.862 85.09 90)
+    (property "Footprint" "Resistor_SMD:R_0402_1005Metric" (at 38.862 85.09 90)
       (effects (font (size 1.27 1.27)) hide)
     )
