File: KiCad7/Hardware_WiRoc_v8/RTC.kicad_sch (KiCad schematic)
At the start: 8 parts, among them U4 74LS73, U9 PCF8563T, Y1 32.768kHz

Commit message: wiroc v8 layout work
Parts:
- R17: footprint Resistor_SMD:R_0603_1608Metric -> Resistor_SMD:R_0402_1005Metric
Changed lines of the file:
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@@
       (effects (font (size 1.27 1.27)) (justify left))
     )
-    (property "Footprint" "Resistor_SMD:R_0603_1608Metric" (at 137.922 72.39 90)
+    (property "Footprint" "Resistor_SMD:R_0402_1005Metric" (at 137.922 72.39 90)
       (effects (font (size 1.27 1.27)) hide)
     )
