File: KiCad7/Hardware_WiRoc_v8/Power1.kicad_sch (KiCad schematic)
At the start: 11 parts, among them Q1 L2N7002WT1G, U18 MP2143DJ

Commit message: more routing of v8
Parts:
- U18: footprint (none) -> WiRoc:TSOT-23-8-Thinner-Pads
Changed lines of the file:
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@@
       (effects (font (size 1.27 1.27)))
     )
-    (property "Footprint" "" (at 121.92 88.9 0)
+    (property "Footprint" "WiRoc:TSOT-23-8-Thinner-Pads" (at 121.92 88.9 0)
       (effects (font (size 1.27 1.27)) hide)
     )
