File: KiCad7/Hardware_WiRoc_v8/Wifi-BT.kicad_sch (KiCad schematic)
At the start: 1 part, among them U19 ESP32-C6-Board

Commit message: more routing of v8
Parts:
- U19: footprint (none) -> WiRoc:ESP32Hosted-C6-Board
Connections:
- net WIFI-UART-CPU_RX: no longer names the net of U19.10 (TXD0)
- net WIFI-UART-CPU_TX: no longer names the net of U19.11 (RXD0)
- no-connect marks 0 -> 2
Changed lines of the file:
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@@
 (kicad_sch (version 20230121) (generator eeschema)
   (paper "A4")
-  (wire (pts (xy 161.29 85.09) (xy 168.91 85.09))
-    (stroke (width 0) (type default))
-  )
-  (wire (pts (xy 161.29 82.55) (xy 168.91 82.55))
-    (stroke (width 0) (type default))
-  )
+  (no_connect (at 161.29 85.09))
+  (no_connect (at 161.29 82.55))
   (global_label "WIFI-SPI-CS0" (shape input) (at 137.16 97.79 180) (fields_autoplaced)
     (effects (font (size 1.524 1.524)) (justify right))
@@
     (property "Intersheetrefs" "${INTERSHEET_REFS}" (at 116.075 85.09 0)
       (effects (font (size 1.27 1.27)) (justify right) hide)
-    )
-  )
-  (global_label "WIFI-UART-CPU_TX" (shape input) (at 168.91 85.09 0) (fields_autoplaced)
-    (effects (font (size 1.524 1.524)) (justify left))
-    (property "Intersheetrefs" "${INTERSHEET_REFS}" (at 193.9862 85.09 0)
-      (effects (font (size 1.27 1.27)) (justify left) hide)
     )
   )
@@
     )
   )
-  (global_label "WIFI-UART-CPU_RX" (shape output) (at 168.91 82.55 0) (fields_autoplaced)
-    (effects (font (size 1.524 1.524)) (justify left))
-    (property "Intersheetrefs" "${INTERSHEET_REFS}" (at 194.3491 82.55 0)
-      (effects (font (size 1.27 1.27)) (justify left) hide)
-    )
-  )
   (symbol (lib_id "WiRoc:ESP32-Hosted-Board") (at 149.86 88.9 0) (unit 1)
     (in_bom yes) (on_board yes) (dnp no)
@@
       (effects (font (size 1.27 1.27)))
     )
-    (property "Footprint" "" (at 149.86 86.36 0)
+    (property "Footprint" "WiRoc:ESP32Hosted-C6-Board" (at 149.86 86.36 0)
       (effects (font (size 1.27 1.27)) hide)
     )
