File: KiCad7/Hardware_WiRoc_v8/eMMC.kicad_sch (KiCad schematic)
At the start: 10 parts, among them U14 KLM8G1WEPD-B031

Commit message: more routing of v8
Connections:
- net GND: now also U14.P2 (NC102)
- net eMMC-CMD: no longer U14.M6 (CLK)
- new net eMMC-CLK: U14.M6 (CLK)
- no-connect marks 111 -> 110
Changed lines of the file:
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@@
   (no_connect (at 160.02 137.16))
   (no_connect (at 121.92 20.32))
-  (no_connect (at 99.06 189.23))
   (no_connect (at 160.02 58.42))
   (no_connect (at 160.02 157.48))
@@
     (effects (font (size 1.524 1.524)) (justify left bottom))
   )
-  (text "*" (at 99.06 193.04 0)
+  (text "*" (at 100.33 193.04 0)
     (effects (font (size 1.524 1.524)) (justify left bottom))
   )
@@
     )
   )
-  (global_label "eMMC-CMD" (shape input) (at 36.83 57.15 180) (fields_autoplaced)
-    (effects (font (size 1.524 1.524)) (justify right))
-    (property "Intersheetrefs" "${INTERSHEET_REFS}" (at 21.0429 57.15 0)
+  (global_label "eMMC-CLK" (shape input) (at 36.83 57.15 180) (fields_autoplaced)
+    (effects (font (size 1.524 1.524)) (justify right))
+    (property "Intersheetrefs" "${INTERSHEET_REFS}" (at 21.5509 57.15 0)
       (effects (font (size 1.27 1.27)) (justify right) hide)
     )
@@
         )
       )
+    )
+  )
+  (symbol (lib_id "power:GND") (at 99.06 189.23 0) (unit 1)
+    (in_bom yes) (on_board yes) (dnp no)
+    (property "Reference" "#PWR0103" (at 99.06 195.58 0)
+      (effects (font (size 1.27 1.27)) hide)
+    )
+    (property "Value" "GND" (at 99.187 193.6242 0)
+      (effects (font (size 1.27 1.27)))
+    )
+    (property "Footprint" "" (at 99.06 189.23 0)
+      (effects (font (size 1.27 1.27)) hide)
+    )
+    (property "Datasheet" "" (at 99.06 189.23 0)
+      (effects (font (size 1.27 1.27)) hide)
+    )
+    (pin "1")
+    (instances
+      (project "WiRoc_NanoPi"
+        (path "/8ba0b499-eaca-4cd5-a002-c6bdb610cc8c/d80ebf4b-5b32-4c39-aa4f-ea56988661f2"
+          (reference "#PWR0103") (unit 1)
+        )
+      )
