File: KiCad9/WiRoc_v8/eMMC.kicad_sch (KiCad schematic)
At the start: 10 parts, among them U14 KLM8G1WEPD-B031

Commit message: many small changes, change eMMC
Parts:
- C66, C67, C71, C83, C84, C85: value 10uF -> 10uF/6.3V
- U14: value KLM8G1WEPD-B031 -> KLM8G1GETF-B041; symbol WiRoc:KLM8G1YEMD-B031 -> WiRoc:KLM8G1GETF-B041; LCSC Part # C2874142 -> C499918; ManufacturerPartNumber KLM8G1WEPD-B031 -> KLM8G1GETF-B041
Connections:
- net eMMC-D7: now also U14.A8 (NC3), U14.B7 (NC11); no longer U14.A7 (RFU1)
- no-connect marks 110 -> 109
Changed lines of the file:
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@@
 	(text "*"
 		(exclude_from_sim no)
+		(at 107.696 17.526 0)
+		(effects
+			(font
+				(size 1.524 1.524)
+			)
+			(justify left bottom)
+		)
+	)
+	(text "*"
+		(exclude_from_sim no)
 		(at 125.73 19.05 0)
 		(effects
@@
 	(text "*"
 		(exclude_from_sim no)
-		(at 100.33 193.04 0)
+		(at 87.884 14.224 0)
 		(effects
 			(font
@@
 	(text "*"
 		(exclude_from_sim no)
-		(at 62.23 76.2 0)
+		(at 100.33 193.04 0)
 		(effects
 			(font
@@
 	)
 	(no_connect
+		(at 72.39 76.2)
+	)
+	(no_connect
 		(at 124.46 189.23)
 	)
@@
 	)
 	(no_connect
-		(at 109.22 20.32)
-	)
-	(no_connect
 		(at 116.84 20.32)
 	)
@@
 	)
 	(no_connect
-		(at 88.9 20.32)
-	)
-	(no_connect
 		(at 160.02 96.52)
 	)
@@
 	(wire
 		(pts
-			(xy 62.23 76.2) (xy 72.39 76.2)
-		)
-		(stroke
-			(width 0)
-			(type default)
-		)
-	)
-	(wire
-		(pts
 			(xy 62.23 36.83) (xy 72.39 36.83)
 		)
@@
 	(wire
 		(pts
-			(xy 106.68 20.32) (xy 106.68 15.24)
+			(xy 106.68 20.32) (xy 106.68 16.51)
 		)
 		(stroke
@@
 	(wire
 		(pts
+			(xy 107.95 13.97) (xy 109.22 13.97)
+		)
+		(stroke
+			(width 0)
+			(type default)
+		)
+	)
+	(wire
+		(pts
 			(xy 31.75 35.56) (xy 35.56 35.56)
 		)
@@
 	(wire
 		(pts
-			(xy 106.68 15.24) (xy 102.87 15.24)
+			(xy 106.68 16.51) (xy 102.87 16.51)
 		)
 		(stroke
@@
 	(wire
 		(pts
+			(xy 109.22 13.97) (xy 109.22 20.32)
+		)
+		(stroke
+			(width 0)
+			(type default)
+		)
+	)
+	(wire
+		(pts
 			(xy 63.5 120.65) (xy 63.5 118.11)
 		)
@@
 	(wire
 		(pts
+			(xy 88.9 19.05) (xy 88.9 20.32)
+		)
+		(stroke
+			(width 0)
+			(type default)
+		)
+	)
+	(wire
+		(pts
 			(xy 63.5 118.11) (xy 72.39 118.11)
 		)
@@
 	(wire
 		(pts
+			(xy 87.63 12.7) (xy 87.63 19.05)
+		)
+		(stroke
+			(width 0)
+			(type default)
+		)
+	)
+	(wire
+		(pts
+			(xy 87.63 19.05) (xy 88.9 19.05)
+		)
+		(stroke
+			(width 0)
+			(type default)
+		)
+	)
+	(wire
+		(pts
 			(xy 66.04 163.83) (xy 66.04 166.37)
 		)
@@
 		)
 	)
+	(global_label "eMMC-D7"
+		(shape bidirectional)
+		(at 107.95 13.97 180)
+		(fields_autoplaced yes)
+		(effects
+			(font
+				(size 1.524 1.524)
+			)
+			(justify right)
+		)
+		(property "Intersheetrefs" "${INTERSHEET_REFS}"
+			(at 92.8342 13.97 0)
+			(effects
+				(font
+					(size 1.27 1.27)
+				)
+				(justify right)
+				(hide yes)
+			)
+		)
+	)
 	(global_label "eMMC-D4"
 		(shape bidirectional)
@@
 	(global_label "eMMC-D3"
 		(shape bidirectional)
-		(at 102.87 15.24 180)
+		(at 102.87 16.51 180)
 		(fields_autoplaced yes)
 		(effects
@@
 		)
 		(property "Intersheetrefs" "${INTERSHEET_REFS}"
-			(at 87.7542 15.24 0)
+			(at 87.7542 16.51 0)
 			(effects
 				(font
@@
 	(global_label "eMMC-D7"
 		(shape bidirectional)
-		(at 62.23 76.2 180)
+		(at 87.63 12.7 180)
 		(fields_autoplaced yes)
 		(effects
@@
 		)
 		(property "Intersheetrefs" "${INTERSHEET_REFS}"
-			(at 47.1142 76.2 0)
+			(at 72.5142 12.7 0)
 			(effects
 				(font
@@
 			)
 		)
-		(property "Value" "10uF"
+		(property "Value" "10uF/6.3V"
 			(at 249.174 83.312 0)
 			(effects
@@
 			)
 		)
-		(property "Value" "10uF"
+		(property "Value" "10uF/6.3V"
 			(at 263.144 52.832 0)
 			(effects
@@
 			)
 		)
-		(property "Value" "10uF"
+		(property "Value" "10uF/6.3V"
 			(at 241.554 52.832 0)
 			(effects
@@
 	)
 	(symbol
-		(lib_id "WiRoc:KLM8G1YEMD-B031")
+		(lib_id "WiRoc:KLM8G1GETF-B041")
 		(at 119.38 110.49 0)
 		(unit 1)
@@
 		(on_board yes)
 		(dnp no)
-		(fields_autoplaced yes)
 		(property "Reference" "U14"
 			(at 152.0541 189.23 0)
@@
 			)
 		)
-		(property "Value" "KLM8G1WEPD-B031"
-			(at 107.95 80.01 0)
+		(property "Value" "KLM8G1GETF-B041"
+			(at 106.934 81.534 0)
 			(effects
 				(font
@@
 			)
 		)
-		(property "Datasheet" ""
+		(property "Datasheet" "https://jlcpcb.com/api/file/downloadByFileSystemAccessId/8588886742133194752"
 			(at 107.95 80.01 0)
 			(effects
@@
 			)
 		)
-		(property "Description" ""
+		(property "Description" "There is also a cheaper alternative: MK MKEV008GCB-SC510 / C2987689"
 			(at 119.38 110.49 0)
 			(effects
@@
 			)
 		)
-		(property "LCSC Part #" "C2874142"
+		(property "LCSC Part #" "C499918"
 			(at 119.38 110.49 0)
 			(effects
@@
 			)
 		)
-		(property "ManufacturerPartNumber" "KLM8G1WEPD-B031"
+		(property "ManufacturerPartNumber" "KLM8G1GETF-B041"
 			(at 119.38 110.49 0)
 			(effects
@@
 			)
 		)
-		(property "Value" "10uF"
+		(property "Value" "10uF/6.3V"
 			(at 230.124 52.832 0)
 			(effects
@@
 			)
 		)
-		(property "Value" "10uF"
+		(property "Value" "10uF/6.3V"
 			(at 260.604 83.312 0)
 			(effects
@@
 			)
 		)
-		(property "Value" "10uF"
+		(property "Value" "10uF/6.3V"
 			(at 251.714 52.832 0)
 			(effects
