File: KiCad9/WiRoc_v8/WiRoc_NanoPi.kicad_sch (KiCad schematic)
At the start: 50 parts, among them J1 Conn_02x05_Odd_Even, J10 Conn_01x09_Socket, J2 Conn_01x04, J5 Conn_01x04_Socket, J6 HAT_Conn_DBG, J8 Conn_01x06, SW1 SW_SPST, U1 SY6280, U10 SY7069ADC, U2 OLED, U3 AXP209, U5 SY6280, U6 BatteryPadM, U7 BatteryPadP

Commit message: many small changes, change eMMC
Parts:
- added R13: 1K, Resistor_SMD:R_0402_1005Metric, symbol Device:R
- C14, C17, C4, C5: value 10uF -> 10uF/6.3V
- R6: value 3.6K-1% -> 10K/1%; footprint Resistor_SMD:R_0603_1608Metric -> Resistor_SMD:R_0402_1005Metric; LCSC Part # C22980 -> C25744; ManufacturerPartNumber 0603WAF3601T5E -> 0402WGF1002TCE; Package 0603 -> 0402
- R9: value 3.6K-1% -> 2K/1%; footprint Resistor_SMD:R_0603_1608Metric -> Resistor_SMD:R_0402_1005Metric; LCSC Part # C22980 -> C4109; ManufacturerPartNumber 0603WAF3601T5E -> 0402WGF2001TCE; Package 0603 -> 0402
Connections:
- net GND: now also R13.1; no longer R9.1
- new net: R13.2, R9.1
Other:
- moved on the sheet: R9
Changed lines of the file:
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@@
 	(wire
 		(pts
-			(xy 262.89 36.83) (xy 262.89 34.29)
-		)
-		(stroke
-			(width 0)
-			(type default)
-		)
-	)
-	(wire
-		(pts
 			(xy 152.4 48.26) (xy 154.94 48.26)
 		)
@@
 			)
 		)
-		(property "Value" "10uF"
+		(property "Value" "10uF/6.3V"
 			(at 269.875 38.1 0)
 			(effects
@@
 	(symbol
 		(lib_id "Device:R")
-		(at 262.89 40.64 180)
+		(at 262.89 38.1 180)
 		(unit 1)
 		(exclude_from_sim no)
@@
 		(dnp no)
 		(property "Reference" "R9"
-			(at 260.858 40.64 90)
+			(at 260.858 38.1 90)
 			(effects
 				(font
@@
 			)
 		)
-		(property "Value" "3.6K-1%"
-			(at 265.43 40.64 90)
+		(property "Value" "2K/1%"
+			(at 265.43 38.1 90)
 			(effects
 				(font
@@
 			)
 		)
-		(property "Footprint" "Resistor_SMD:R_0603_1608Metric"
-			(at 264.668 40.64 90)
+		(property "Footprint" "Resistor_SMD:R_0402_1005Metric"
+			(at 264.668 38.1 90)
 			(effects
 				(font
@@
 		)
 		(property "Datasheet" "~"
-			(at 262.89 40.64 0)
+			(at 262.89 38.1 0)
 			(effects
 				(font
@@
 		)
 		(property "Description" ""
-			(at 262.89 40.64 0)
+			(at 262.89 38.1 0)
 			(effects
 				(font
@@
 			)
 		)
-		(property "Package" "0603"
-			(at 262.89 40.64 90)
+		(property "Package" "0402"
+			(at 262.89 38.1 90)
 			(effects
 				(font
@@
 			)
 		)
-		(property "ManufacturerPartNumber" "0603WAF3601T5E"
-			(at 262.89 40.64 90)
+		(property "ManufacturerPartNumber" "0402WGF2001TCE"
+			(at 262.89 38.1 90)
 			(effects
 				(font
@@
 		)
 		(property "Original" "No"
-			(at 262.89 40.64 90)
+			(at 262.89 38.1 90)
 			(effects
 				(font
@@
 		)
 		(property "Manufacturer" "Uniroyal Elec"
-			(at 525.78 -6.35 0)
+			(at 525.78 -8.89 0)
 			(effects
 				(font
@@
 		)
 		(property "WebsiteURL" "https://lcsc.com/product-detail/Chip-Resistor-Surface-Mount_3-6KR-3601-1_C100993.html"
-			(at 525.78 -6.35 0)
+			(at 525.78 -8.89 0)
 			(effects
 				(font
@@
 		)
 		(property "IncludeInBOM" "TRUE"
-			(at 262.89 40.64 90)
+			(at 262.89 38.1 90)
 			(effects
 				(font
@@
 		)
 		(property "ThroughHole" "FALSE"
-			(at 525.78 -6.35 0)
+			(at 525.78 -8.89 0)
 			(effects
 				(font
@@
 			)
 		)
-		(property "LCSC Part #" "C22980"
-			(at 262.89 40.64 0)
+		(property "LCSC Part #" "C4109"
+			(at 262.89 38.1 0)
 			(effects
 				(font
@@
 		)
 		(property "JLCPCB Rotation Offset" ""
-			(at 262.89 40.64 0)
+			(at 262.89 38.1 0)
 			(effects
 				(font
@@
 		)
 		(property "JLCBasicExtended" "Basic"
-			(at 262.89 40.64 90)
+			(at 262.89 38.1 90)
 			(effects
 				(font
@@
 	(symbol
 		(lib_id "power:GND")
-		(at 262.89 44.45 0)
+		(at 262.89 49.53 0)
 		(unit 1)
 		(exclude_from_sim no)
@@
 		(dnp no)
 		(property "Reference" "#PWR06"
-			(at 262.89 50.8 0)
+			(at 262.89 55.88 0)
 			(effects
 				(font
@@
 		)
 		(property "Value" "GND"
-			(at 262.89 48.26 0)
+			(at 262.89 53.34 0)
 			(effects
 				(font
@@
 		)
 		(property "Footprint" ""
-			(at 262.89 44.45 0)
+			(at 262.89 49.53 0)
 			(effects
 				(font
@@
 		)
 		(property "Datasheet" ""
-			(at 262.89 44.45 0)
+			(at 262.89 49.53 0)
 			(effects
 				(font
@@
 		)
 		(property "Description" ""
-			(at 262.89 44.45 0)
+			(at 262.89 49.53 0)
 			(effects
 				(font
@@
 			)
 		)
-		(property "Value" "10uF"
+		(property "Value" "10uF/6.3V"
 			(at 44.45 89.535 0)
 			(effects
@@
 			)
 		)
-		(property "Value" "10uF"
+		(property "Value" "10uF/6.3V"
 			(at 45.72 107.315 0)
 			(effects
@@
 			)
 		)
-		(property "Value" "3.6K-1%"
+		(property "Value" "10K/1%"
 			(at 126.492 41.148 90)
 			(effects
@@
 			)
 		)
-		(property "Footprint" "Resistor_SMD:R_0603_1608Metric"
+		(property "Footprint" "Resistor_SMD:R_0402_1005Metric"
 			(at 126.238 40.64 90)
 			(effects
@@
 			)
 		)
-		(property "Package" "0603"
+		(property "Package" "0402"
 			(at 124.46 40.64 90)
 			(effects
@@
 			)
 		)
-		(property "ManufacturerPartNumber" "0603WAF3601T5E"
+		(property "ManufacturerPartNumber" "0402WGF1002TCE"
 			(at 124.46 40.64 90)
 			(effects
@@
 			)
 		)
-		(property "LCSC Part #" "C22980"
+		(property "LCSC Part #" "C25744"
 			(at 124.46 40.64 0)
 			(effects
@@
 			)
 		)
-		(property "Value" "10uF"
+		(property "Value" "10uF/6.3V"
 			(at 123.444 33.782 0)
 			(effects
@@
 					(unit 1)
 				)
+			)
+		)
+	)
+	(symbol
+		(lib_id "Device:R")
+		(at 262.89 45.72 180)
+		(unit 1)
+		(exclude_from_sim no)
+		(in_bom yes)
+		(on_board yes)
+		(dnp no)
+		(property "Reference" "R13"
+			(at 260.858 45.72 90)
+			(effects
+				(font
+					(size 1.27 1.27)
+				)
+			)
+		)
+		(property "Value" "1K"
+			(at 265.43 45.72 90)
+			(effects
+				(font
+					(size 1.27 1.27)
+				)
+			)
+		)
+		(property "Footprint" "Resistor_SMD:R_0402_1005Metric"
+			(at 264.668 45.72 90)
+			(effects
+				(font
+					(size 1.27 1.27)
+				)
+				(hide yes)
+			)
+		)
+		(property "Datasheet" "~"
+			(at 262.89 45.72 0)
+			(effects
+				(font
+					(size 1.27 1.27)
+				)
+				(hide yes)
+			)
+		)
+		(property "Description" "1KΩ (1001) ±1%"
+			(at 262.89 45.72 0)
+			(effects
+				(font
+					(size 1.27 1.27)
+				)
+				(hide yes)
+			)
+		)
+		(property "Package" "0402"
+			(at 262.89 45.72 90)
+			(effects
+				(font
+					(size 1.524 1.524)
+				)
+				(hide yes)
+			)
+		)
+		(property "ManufacturerPartNumber" "0402WGF1001TCE"
+			(at 262.89 45.72 90)
+			(effects
+				(font
+					(size 1.524 1.524)
+				)
+				(hide yes)
+			)
+		)
+		(property "Original" "No"
+			(at 262.89 45.72 90)
+			(effects
+				(font
+					(size 1.524 1.524)
+				)
+				(hide yes)
+			)
+		)
+		(property "Manufacturer" "Uniroyal Elec"
+			(at 525.78 -1.27 0)
+			(effects
+				(font
+					(size 1.27 1.27)
+				)
+				(hide yes)
+			)
+		)
+		(property "WebsiteURL" "https://lcsc.com/product-detail/Chip-Resistor-Surface-Mount_3-6KR-3601-1_C100993.html"
+			(at 525.78 -1.27 0)
+			(effects
+				(font
+					(size 1.27 1.27)
+				)
+				(hide yes)
+			)
+		)
+		(property "IncludeInBOM" "TRUE"
+			(at 262.89 45.72 90)
+			(effects
+				(font
+					(size 1.27 1.27)
+				)
+				(hide yes)
+			)
+		)
+		(property "ThroughHole" "FALSE"
+			(at 525.78 -1.27 0)
+			(effects
+				(font
+					(size 1.27 1.27)
+				)
+				(hide yes)
+			)
+		)
+		(property "LCSC Part #" "C11702"
+			(at 262.89 45.72 0)
+			(effects
+				(font
+					(size 1.27 1.27)
+				)
+				(hide yes)
+			)
+		)
+		(property "JLCPCB Rotation Offset" ""
+			(at 262.89 45.72 0)
+			(effects
+				(font
+					(size 1.27 1.27)
+				)
+				(hide yes)
+			)
+		)
+		(property "JLCBasicExtended" "Basic"
+			(at 262.89 45.72 90)
+			(effects
+				(font
+					(size 1.27 1.27)
+				)
+				(hide yes)
+			)
+		)
+		(pin "1"
+		)
+		(pin "2"
+		)
+		(instances
+			(project "WiRoc_NanoPi"
+				(path "/8ba0b499-eaca-4cd5-a002-c6bdb610cc8c"
+					(reference "R13")
+					(unit 1)
+				)

Commit message: etc
Parts:
- J1, J10, J5: now left out of the parts list
- U1, U5: FT Rotation Offset (none) -> 90; JLCPCB Rotation Offset -90 -> (none)
- U10: FT Rotation Offset (none) -> 0; JLCPCB Rotation Offset 180 -> (none)

Commit message: add ethernet etc
Parts:
- removed J1: Conn_02x05_Odd_Even, Connector_PinHeader_1.27mm:PinHeader_2x05_P1.27mm_Vertical, symbol Connector_Generic:Conn_02x05_Odd_Even
- added J12: TC2050, Connector:Tag-Connect_TC2050-IDC-NL_2x05_P1.27mm_Vertical, symbol Connector:TC2050
- J2: footprint Connector_PinHeader_1.27mm:PinHeader_1x04_P1.27mm_Horizontal -> WiRoc:PinSocket_1x04_P1.27mm_RightAngled
- J8: footprint Connector_PinHeader_1.27mm:PinHeader_1x06_P1.27mm_Horizontal -> WiRoc:PinSocket_1x06_P1.27mm_RightAngled
Connections:
- net GND: now also J12.2, J12.3
- net SRR_NRST: now also J12.6
- net VDD_SRR: now also J12.1
- net at J2.1 (Pin_1): now also J12.9
- net at J2.2 (Pin_2): now also J12.4
- net at J2.3 (Pin_3): now also J12.5
- net at J8.4 (Pin_4): now also J12.10
Changed lines of the file:
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@@
 	)
 	(symbol
+		(lib_name "GND_1")
 		(lib_id "power:GND")
 		(at 105.41 86.36 90)
@@
 			)
 		)
-		(property "Description" ""
+		(property "Description" "Power symbol creates a global label with name \"GND\" , ground"
 			(at 105.41 86.36 0)
 			(effects
@@
 			)
 		)
-		(property "Footprint" "Connector_PinHeader_1.27mm:PinHeader_1x04_P1.27mm_Horizontal"
+		(property "Footprint" "WiRoc:PinSocket_1x04_P1.27mm_RightAngled"
 			(at 160.02 45.72 0)
 			(effects
@@
 	)
 	(symbol
+		(lib_id "Connector:TC2050")
+		(at 144.78 38.1 180)
+		(unit 1)
+		(exclude_from_sim no)
+		(in_bom no)
+		(on_board yes)
+		(dnp no)
+		(fields_autoplaced yes)
+		(property "Reference" "J12"
+			(at 143.51 22.86 0)
+			(effects
+				(font
+					(size 1.27 1.27)
+				)
+			)
+		)
+		(property "Value" "TC2050"
+			(at 143.51 25.4 0)
+			(effects
+				(font
+					(size 1.27 1.27)
+				)
+			)
+		)
+		(property "Footprint" "Connector:Tag-Connect_TC2050-IDC-NL_2x05_P1.27mm_Vertical"
+			(at 143.51 38.1 0)
+			(effects
+				(font
+					(size 1.27 1.27)
+				)
+				(hide yes)
+			)
+		)
+		(property "Datasheet" "https://www.tag-connect.com/wp-content/uploads/bsk-pdf-manager/TC2050-IDC-NL_Datasheet_8.pdf"
+			(at 143.51 38.1 0)
+			(effects
+				(font
+					(size 1.27 1.27)
+				)
+				(hide yes)
+			)
+		)
+		(property "Description" "Tag-Connect’s 10-pins connector"
+			(at 144.78 38.1 0)
+			(effects
+				(font
+					(size 1.27 1.27)
+				)
+				(hide yes)
+			)
+		)
+		(pin "6"
+		)
+		(pin "5"
+		)
+		(pin "4"
+		)
+		(pin "1"
+		)
+		(pin "9"
+		)
+		(pin "2"
+		)
+		(pin "3"
+		)
+		(pin "10"
+		)
+		(pin "7"
+		)
+		(pin "8"
+		)
+		(instances
+			(project ""
+				(path "/8ba0b499-eaca-4cd5-a002-c6bdb610cc8c"
+					(reference "J12")
+					(unit 1)
+				)
+			)
+		)
+	)
+	(symbol
 		(lib_id "power:GND")
 		(at 113.03 44.45 0)
@@
 			)
 		)
-		(property "Footprint" "Connector_PinHeader_1.27mm:PinHeader_1x06_P1.27mm_Horizontal"
+		(property "Footprint" "WiRoc:PinSocket_1x06_P1.27mm_RightAngled"
 			(at 160.02 19.05 0)
 			(effects
@@
 					(unit 1)
 				)
-			)
-		)
-	)
-	(symbol
-		(lib_id "Connector_Generic:Conn_02x05_Odd_Even")
-		(at 144.78 38.1 180)
-		(unit 1)
-		(exclude_from_sim no)
-		(in_bom no)
-		(on_board yes)
-		(dnp no)
-		(property "Reference" "J1"
-			(at 138.43 46.99 0)
-			(effects
-				(font
-					(size 1.27 1.27)
-				)
-			)
-		)
-		(property "Value" "Conn_02x05_Odd_Even"
-			(at 144.78 29.21 0)
-			(effects
-				(font
-					(size 1.27 1.27)
-				)
-			)
-		)
-		(property "Footprint" "Connector_PinHeader_1.27mm:PinHeader_2x05_P1.27mm_Vertical"
-			(at 144.78 38.1 0)
-			(effects
-				(font
-					(size 1.27 1.27)
-				)
-				(hide yes)
-			)
-		)
-		(property "Datasheet" "~"
-			(at 144.78 38.1 0)
-			(effects
-				(font
-					(size 1.27 1.27)
-				)
-				(hide yes)
-			)
-		)
-		(property "Description" ""
-			(at 144.78 38.1 0)
-			(effects
-				(font
-					(size 1.27 1.27)
-				)
-				(hide yes)
-			)
-		)
-		(property "JLCBasicExtended" "Extended"
-			(at 144.78 38.1 0)
-			(effects
-				(font
-					(size 1.27 1.27)
-				)
-				(hide yes)
-			)
-		)
-		(property "IncludeInBOM" "FALSE"
-			(at 144.78 38.1 0)
-			(effects
-				(font
-					(size 1.27 1.27)
-				)
-				(hide yes)
-			)
-		)
-		(property "LCSC Part #" "C5142394"
-			(at 144.78 38.1 0)
-			(effects
-				(font
-					(size 1.27 1.27)
-				)
-				(hide yes)
-			)
-		)
-		(property "Manufacturer" "MINTRON"
-			(at 144.78 38.1 0)
-			(effects
-				(font
-					(size 1.27 1.27)
-				)
-				(hide yes)
-			)
-		)
-		(property "ManufacturerPartNumber" "MTP310-1205S2"
-			(at 144.78 38.1 0)
-			(effects
-				(font
-					(size 1.27 1.27)
-				)
-				(hide yes)
-			)
-		)
-		(pin "1"
-		)
-		(pin "10"
-		)
-		(pin "2"
-		)
-		(pin "3"
-		)
-		(pin "4"
-		)
-		(pin "5"
-		)
-		(pin "6"
-		)
-		(pin "7"
-		)
-		(pin "8"
-		)
-		(pin "9"
-		)
-		(instances
-			(project "WiRoc_NanoPi"
-				(path "/8ba0b499-eaca-4cd5-a002-c6bdb610cc8c"
-					(reference "J1")
-					(unit 1)
-				)
