File: KiCad9/SRRReceiver_v5/SRRReceiver.kicad_sch (KiCad schematic)
At the start: 51 parts, among them J2 Conn_01x06, J3 Conn_01x04, U1 CC2500, U2 CC2500, U3 STM32G071KxT, Y1 Crystal_GND24 Cload=10pF 26MHz, Y2 Crystal_GND24 Cload=10pF 26MHz

Commit message: etc
Parts:
- removed C2, C22: 47pF, Capacitor_SMD:C_0402_1005Metric, symbol Device:C
- removed C24, C25, C3, C4: 220pF, Capacitor_SMD:C_0402_1005Metric, symbol Device:C
- removed C8: 100nF, Capacitor_SMD:C_0402_1005Metric, symbol Device:C
- C1, C5, C6: value 100nF -> 10uF; LCSC C1525 -> C15525
- C11, C23: value 220pF -> 10uF; LCSC C16772 -> C15525
- C21, C26, C27: value 0.1uF -> 10uF; LCSC C1525 -> C15525
- C9: value 4.7nF -> 10uF; LCSC C1538 -> C15525
