File: KiCad9/SRRReceiver_v5/SRRReceiver.kicad_pcb (KiCad board)
At the start: 4 copper layers, 28.6 x 24.1 mm, 51 parts, among them J2 Conn_01x06, J3 Conn_01x04, U1 CC2500, U2 CC2500, U3 STM32G071KxT, Y1 Crystal_GND24 Cload=10pF 26MHz, Y2 Crystal_GND24 Cload=10pF 26MHz

Commit message: etc
Parts:
- removed C2, C22: 47pF, Capacitor_SMD:C_0402_1005Metric
- removed C24, C25, C3, C4: 220pF, Capacitor_SMD:C_0402_1005Metric
- removed C8: 100nF, Capacitor_SMD:C_0402_1005Metric
- C1, C5, C6: value 100nF -> 10uF
- C11, C23: value 220pF -> 10uF
- C21, C26, C27: value 0.1uF -> 10uF
- C9: value 4.7nF -> 10uF
- moved C9 0.91 mm to (129.2, 89.0)
- moved C1 0.74 mm to (129.8, 94.5)
- moved C21 0.49 mm to (118.9, 84.3)
- moved C28 0.47 mm to (119.0, 86.4)
- moved C27 0.36 mm to (123.3, 86.9)
- moved C12 0.28 mm to (129.3, 92.2)
- moved C6 0.16 mm to (125.4, 91.7)
- moved C11 0.16 mm to (126.9, 98.2)
- moved R1 0.15 mm to (125.0, 98.2)
- moved C23 0.14 mm to (121.8, 80.7)
- moved R2 0.14 mm to (123.7, 80.7)
- moved C5 0.11 mm to (123.5, 98.0)
- moved C7 0.11 mm to (128.2, 90.2)
- moved C18 0.11 mm to (120.5, 88.9)
Routing:
- net VDD: track 35.0 -> 27.6 mm
- net GND: track 30.6 -> 27.1 mm, vias 111 -> 120
- net SPI1_MISO: track 10.9 -> 10.2 mm
- net SPI1_SCK: track 12.3 -> 11.7 mm

Commit message: add ethernet etc
Other:
- board text added: "10uF"
- board text removed: "100nF"
- board text removed: "4.7nF"
Changed lines of the file:
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@@
 		)
 		(embedded_fonts no)
-		(model "${KICAD6_3DMODEL_DIR}/Package_DFN_QFN.3dshapes/Texas_S-PVQFN-N20_EP2.4x2.4mm.wrl"
+		(model "${KICAD9_3DMODEL_DIR}/Package_DFN_QFN.3dshapes/Texas_S-PWQFN-N20.wrl"
 			(offset
 				(xyz 0 0 0)
@@
 		)
 		(embedded_fonts no)
-		(model "${KICAD6_3DMODEL_DIR}/Package_DFN_QFN.3dshapes/Texas_S-PVQFN-N20_EP2.4x2.4mm.wrl"
+		(model "${KICAD9_3DMODEL_DIR}/Package_DFN_QFN.3dshapes/Texas_S-PWQFN-N20.wrl"
 			(offset
 				(xyz 0 0 0)
@@
 		)
 		(embedded_fonts no)
-		(model "${KICAD6_3DMODEL_DIR}/Connector_PinSocket_1.27mm.3dshapes/PinSocket_1x04_P1.27mm_Vertical.wrl"
+		(model "${KICAD9_3DMODEL_DIR}/Connector_PinHeader_1.27mm.3dshapes/PinHeader_1x04_P1.27mm_Vertical.wrl"
 			(offset
 				(xyz 0 0 0)
@@
 		)
 		(embedded_fonts no)
-		(model "${KICAD6_3DMODEL_DIR}/Connector_PinSocket_1.27mm.3dshapes/PinSocket_1x06_P1.27mm_Vertical.wrl"
+		(model "${KICAD9_3DMODEL_DIR}/Connector_PinHeader_1.27mm.3dshapes/PinHeader_1x06_P1.27mm_Vertical.wrl"
 			(offset
 				(xyz 0 0 0)
@@
 		)
 	)
-	(gr_text "4.7nF"
-		(at 128.8 87.8 315)
-		(layer "B.SilkS")
-		(effects
-			(font
-				(size 0.6 0.6)
-				(thickness 0.15)
-				(bold yes)
-			)
-			(justify left bottom mirror)
-		)
-	)
-	(gr_text "100nF"
-		(at 128.2 88.4 -45)
+	(gr_text "10uF"
+		(at 128.1 88.47 315)
 		(layer "B.SilkS")
 		(effects
