File: KiCad10/WiRoc_v8/WiRoc_NanoPi.kicad_pcb (KiCad board)
At the start: 6 copper layers, 48 x 68.7 mm, 196 parts, among them J1 TC2050, J10 Conn_01x09_Socket, J11 Conn_01x05, J12 TC2050, J2 Conn_01x04, J3 Micro_SD_Card_Det1, J4 Conn_01x09_Socket, J5 Conn_01x04_Socket, J6 HAT_Conn_DBG, J8 Conn_01x06, J9 Conn_Coaxial, Q1 L2N7002WT1G, SW1 SW_SPST, SW2 SW_SPST, U1 SY6280, U10 SY7069ADC, U11 AllwinnerH3, U12 DDR3, U13 SGM803-RXN3L, U14 KLM8G1GETF-B041, U15 RT8059, U16 RT8059, U17 RT8059, U18 MP2143DJ, U19 ESP32-C5-Board, U2 OLED, U20 SY6280, U3 AXP209, U4 74HC73, U5 SY6280, U6 BatteryPadM, U7 BatteryPadP, U8 RAK3172-xx-43-SM-xI, U9 PCF8563T, Y1 32.768kHz, Y2 24MHz/CL=12pF

Commit message: kicad10 and .gitignore lck history
Routing:
- net eMMC-D2: track 19.1 -> 13.3 mm
- net eMMC-D1: track 16.8 -> 12.8 mm
- net WIFI-SPI-SCLK: track 50.4 -> 53.3 mm
- net eMMC-D6: track 17.1 -> 14.6 mm
- net eMMC-D0: track 17.6 -> 19.9 mm
- net eMMC-D3: track 18.1 -> 20.3 mm
- net WIFI-SPI-MOSI: track 52.0 -> 54.1 mm
- net eMMC-D5: track 18.0 -> 19.9 mm
- net eMMC-D7: track 17.0 -> 15.2 mm
- net /Processor-MEM/SA3: track 18.1 -> 19.7 mm
- net eMMC-D4: track 15.8 -> 17.2 mm
- net SDQ7: track 15.2 -> 14.0 mm
- net /Processor-MEM/SA10: track 15.4 -> 16.4 mm
- net /Processor-MEM/SA9: track 14.7 -> 15.6 mm
- net /Processor-MEM/SA4: track 18.1 -> 19.0 mm
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