File: KiCad10/WiRoc_v8/LED-Etc.kicad_sch (KiCad schematic)
At the start: 4 parts

Commit message: add logo, improve layout
Parts:
- R39, R41: ManufacturerPartNumber 0402WGF1001TCE -> 0402WGF2001TCE
- R40: ManufacturerPartNumber 0402WGF1001TCE -> 0402WGF1002TCE
Changed lines of the file:
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@@
 (kicad_sch
-	(version 20260326)
+	(version 20260306)
 	(generator "eeschema")
-	(generator_version "10.99")
+	(generator_version "10.0")
 	(paper "A4")
 	(junction
@@
 			)
 		)
-		(property "Description" "1KΩ (1001) ±1%"
+		(property "Description" ""
 			(at 88.9 55.88 90)
 			(hide yes)
@@
 			)
 		)
-		(property "ManufacturerPartNumber" "0402WGF1001TCE"
+		(property "ManufacturerPartNumber" "0402WGF2001TCE"
 			(at 88.9 55.88 90)
 			(hide yes)
@@
 			)
 		)
-		(property "Description" "1KΩ (1001) ±1%"
+		(property "Description" ""
 			(at 80.01 40.64 90)
 			(hide yes)
@@
 			)
 		)
-		(property "ManufacturerPartNumber" "0402WGF1001TCE"
+		(property "ManufacturerPartNumber" "0402WGF1002TCE"
 			(at 80.01 40.64 90)
 			(hide yes)
@@
 			)
 		)
-		(property "Description" "1KΩ (1001) ±1%"
+		(property "Description" ""
 			(at 88.9 50.8 90)
 			(hide yes)
@@
 			)
 		)
-		(property "ManufacturerPartNumber" "0402WGF1001TCE"
+		(property "ManufacturerPartNumber" "0402WGF2001TCE"
 			(at 88.9 50.8 90)
 			(hide yes)
