File: KiCad10/WiRoc_v8/LED-Etc.kicad_sch (KiCad schematic)
At the start: 4 parts

Commit message: fix rotation of LED
Parts:
- D2: FT Rotation Offset (none) -> 180
Changed lines of the file:
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@@
 			)
 		)
-		(property "FT Rotation Offset" ""
+		(property "FT Rotation Offset" "180"
 			(at 105.41 53.34 0)
 			(hide yes)
