File: KiCad10/WiRoc_v8/Power2.kicad_sch (KiCad schematic)
At the start: 23 parts, among them U15 RT8059, U16 RT8059, U17 RT8059

Commit message: add logo, improve layout
Parts:
- L2, L4, L5: LCSC Part # C882952 -> C576403
Changed lines of the file:
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@@
 (kicad_sch
-	(version 20260326)
+	(version 20260306)
 	(generator "eeschema")
-	(generator_version "10.99")
+	(generator_version "10.0")
 	(paper "A4")
 	(text "Vfb=0.6V"
@@
 			)
 		)
-		(property "Description" ""
+		(property "Description" "2.2uH 2.3A 3.6A 82mΩ ±20% 1008 Power Inductors ROHS"
 			(at 127 118.11 0)
 			(hide yes)
@@
 			)
 		)
-		(property "LCSC Part #" "C882952"
+		(property "LCSC Part #" "C576403"
 			(at 127 118.11 90)
 			(hide yes)
@@
 			)
 		)
-		(property "Description" ""
+		(property "Description" "2.2uH 2.3A 3.6A 82mΩ ±20% 1008 Power Inductors ROHS"
 			(at 127 72.39 0)
 			(hide yes)
@@
 			)
 		)
-		(property "LCSC Part #" "C882952"
+		(property "LCSC Part #" "C576403"
 			(at 127 72.39 90)
 			(hide yes)
@@
 			)
 		)
-		(property "Description" ""
+		(property "Description" "2.2uH 2.3A 3.6A 82mΩ ±20% 1008 Power Inductors ROHS"
 			(at 127 26.67 0)
 			(hide yes)
@@
 			)
 		)
-		(property "LCSC Part #" "C882952"
+		(property "LCSC Part #" "C576403"
 			(at 127 26.67 90)
 			(hide yes)

Commit message: etc
Parts:
- R49: LCSC Part # C25157 -> C270630; ManufacturerPartNumber 0402WGJ020JTCE -> 0402WGF200KTCE
Changed lines of the file:
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@@
 			)
 		)
-		(property "LCSC Part #" "C25157"
+		(property "LCSC Part #" "C270630"
 			(at 172.72 118.11 90)
 			(hide yes)
@@
 			)
 		)
-		(property "ManufacturerPartNumber" "0402WGJ020JTCE"
+		(property "ManufacturerPartNumber" "0402WGF200KTCE"
 			(at 172.72 118.11 90)
 			(hide yes)
