File: KiCad10/WiRoc_v8/Power2.kicad_sch (KiCad schematic)
At the start: 23 parts, among them U15 RT8059, U16 RT8059, U17 RT8059

Commit message: change partnumber
Parts:
- R49: LCSC Part # C270630 -> C2998051; Manufacturer Uniroyal Elec -> Fojan; ManufacturerPartNumber 0402WGF200KTCE -> FRC0402F2R00TS
Changed lines of the file:
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@@
 			)
 		)
-		(property "LCSC Part #" "C270630"
+		(property "LCSC Part #" "C2998051"
 			(at 172.72 118.11 90)
 			(hide yes)
@@
 			)
 		)
-		(property "Manufacturer" "Uniroyal Elec"
+		(property "Manufacturer" "Fojan"
 			(at 172.72 118.11 90)
 			(hide yes)
@@
 			)
 		)
-		(property "ManufacturerPartNumber" "0402WGF200KTCE"
+		(property "ManufacturerPartNumber" "FRC0402F2R00TS"
 			(at 172.72 118.11 90)
 			(hide yes)
