File: KiCad10/WiRoc_v8/RTC.kicad_sch (KiCad schematic)
At the start: 8 parts, among them U4 74HC73, U9 PCF8563T, Y1 32.768kHz

Commit message: etc
Connections:
- no-connect marks 5 -> 3
Changed lines of the file:
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@@
-	)
-	(no_connect
-		(at 232.41 40.64)
 	)
 	(no_connect
@@
 	)
 	(no_connect
-		(at 233.68 40.64)
-	)
-	(no_connect
