File: KiCad10/WiRoc_v8/Lora.kicad_sch (KiCad schematic)
At the start: 17 parts, among them J1 TC2050, J11 Conn_01x05, J9 Conn_Coaxial, SW2 SW_SPST, U20 SY6280, U8 RAK3172-xx-43-SM-xI

Commit message: fix rotation of LED
Parts:
- D3: FT Rotation Offset (none) -> 180
Changed lines of the file:
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@@
 			)
 		)
-		(property "FT Rotation Offset" ""
+		(property "FT Rotation Offset" "180"
 			(at 200.66 88.9 0)
 			(hide yes)
