File: KiCad10/NanoPi_v8_USBConnectorPlate/Hardware_NanoPi_v8_USBConnectorPlate.kicad_pcb (KiCad board)
At the start: 2 copper layers, 16 x 60 mm, 48 parts, among them J1 Conn_01x02, J10 Conn_01x04, J11 Conn_01x02, J12 Conn_01x02, J2 USB_Host_Data_02x02, J3 USB_Host_Data_02x02, J4 USB_Power_02x02, J5 Conn_01x05, J6 Conn_01x09, J8 Conn_01x09, U1 USBLC6-2P6, U2 USBLC6-2P6, U3 USBLC6-2P6, U4 ALT4532M-201-T001, U5 ALT4532M-201-T001, U8 SP3232ECY-L

Commit message: etc
Parts:
- C10, C11, C7, C8, C9: value 100nF -> 100 nF

Commit message: etc
Parts:
- U4, U5: value ALT4532M-201-T001 -> ALT4532M-170-T001
- moved U1 9.85 mm to (115.8, 88.5)
- moved U2 5.97 mm to (111.9, 75.8)
- moved J3 0.07 mm to (110.5, 90.0)
Connections:
- net Net-(J2-Pin_2) renamed /USB1-DM-ToPad
- net Net-(J2-Pin_3) renamed /USB1-DP-ToPad
- net Net-(J3-Pin_2) renamed /USB2-DM-ToPad
- net Net-(J3-Pin_3) renamed /USB2-DP-ToPad
- FL3 pad 1: Net-(FL3-Pad1) -> /USB1-DP-ToESD
- FL3 pad 2: Net-(FL3-Pad2) -> /USB1-DM-ToESD
- FL3 pad 3: USBHost-DP1 -> USBHost-DM1
- FL3 pad 4: USBHost-DM1 -> USBHost-DP1
- FL4 pad 1: Net-(FL4-Pad1) -> /USB2-DP-ToESD
- FL4 pad 2: Net-(FL4-Pad2) -> /USB2-DM-ToESD
- FL4 pad 3: USBHost-DP2 -> USBHost-DM2
- FL4 pad 4: USBHost-DM2 -> USBHost-DP2
- U1 pad 4: Net-(FL4-Pad2) -> /USB2-DP-ToESD
- U1 pad 6: Net-(FL4-Pad1) -> /USB2-DM-ToESD
- U2 pad 4: Net-(FL3-Pad2) -> /USB1-DP-ToESD
- U2 pad 6: Net-(FL3-Pad1) -> /USB1-DM-ToESD
Routing:
- net /USB2-DM-ToPad: track 13.9 -> 2.59 mm
- net /USB2-DP-ToESD: track 0.00 -> 10.9 mm
- net /USB2-DM-ToESD: track 0.00 -> 8.56 mm
- net /USB1-DP-ToPad: track 10.4 -> 2.88 mm
- net /USB1-DM-ToESD: track 0.00 -> 5.89 mm
- net Net-(FL3-Pad2): track 3.76 -> 0.00 mm
- net /USB1-DP-ToESD: track 0.00 -> 3.65 mm
- net Net-(FL4-Pad1): track 3.47 -> 0.00 mm
- net GND: track 16.3 -> 13.3 mm, vias 44 -> 47
- net /USB2-DP-ToPad: track 6.76 -> 4.45 mm
- net VDD_5V_OUT2: track 19.0 -> 21.1 mm
- net Net-(FL3-Pad1): track 1.77 -> 0.00 mm
- net Net-(FL4-Pad2): track 1.61 -> 0.00 mm
- net /USB1-DM-ToPad: track 3.52 -> 4.85 mm
- net USBHost-DP1: track 3.79 -> 3.31 mm, vias 1 -> 0
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