File: KiCad10/NanoPi_v8_USBConnectorPlate/Hardware_NanoPi_v8_USBConnectorPlate.kicad_sch (KiCad schematic)
At the start: 48 parts, among them J1 Conn_01x02, J10 Conn_01x04, J11 Conn_01x02, J12 Conn_01x02, J2 USB_Host_Data_02x02, J3 USB_Host_Data_02x02, J4 USB_Power_02x02, J5 Conn_01x05, J6 Conn_01x09, J8 Conn_01x09, U1 USBLC6-2P6, U2 USBLC6-2P6, U3 USBLC6-2P6, U4 ALT4532M-201-T001, U5 ALT4532M-201-T001, U8 SP3232ECY-L

Commit message: etc
Parts:
- C1, C2, C3, C4, C5, C6, R1, R2, R3, R4, R5, R6: Basic (none) -> YES
- C10, C11, C7, C8, C9: Basic (none) -> YES; IncludeInBOM TRUE -> (none)
- C12, C13, C14, R7, R8: Basic (none) -> YES; now not fitted; now left out of the parts list
- FB1, FB2, FB3, FL3, FL4, U1, U2, U3: Basic (none) -> NO
- FB4, FL1, FL2: Basic (none) -> NO; now not fitted; now left out of the parts list
- J1, J10, J11, J12, J5, J6, J8: now left out of the parts list
- J2, J3, J4: IncludeInBOM FALSE -> (none)
- U4, U5: value ALT4532M-201-T001 -> ALT4532M-170-T001; Basic (none) -> NO; now not fitted; now left out of the parts list
- U8: Basic (none) -> NO; IncludeInBOM TRUE -> (none)

Commit message: etc
Parts:
- C7: LCSC C307331 -> C1525; LCSC Part # C307331 -> C1525
Connections:
- net USBHost-DM1: now also FL3.3; no longer FL3.4
- net USBHost-DM2: now also FL4.3; no longer FL4.4
- net USBHost-DP1: now also FL3.4; no longer FL3.3
- net USBHost-DP2: now also FL4.4; no longer FL4.3
- net USB1-DM-ToPad: now reaches J2.2 (Pin_2), U2.1 (I/O1)
- net USB1-DP-ToPad: now reaches J2.3 (Pin_3), U2.3 (I/O2)
- net USB2-DM-ToPad: now reaches J3.2 (Pin_2), U1.1 (I/O1)
- net USB2-DP-ToPad: now reaches J3.3 (Pin_3), U1.3 (I/O2)
- net USB2-DM-ToESD: now reaches FL4.2
- net USB2-DM-ToESD: now also U1.6 (I/O1); no longer U1.4 (I/O2)
- net USB2-DP-ToESD: now reaches FL4.1
- net USB2-DP-ToESD: now also U1.4 (I/O2); no longer U1.6 (I/O1)
- net USB1-DM-ToESD: now reaches FL3.2
- net USB1-DM-ToESD: now also U2.6 (I/O1); no longer U2.4 (I/O2)
- net USB1-DP-ToESD: now reaches FL3.1
- net USB1-DP-ToESD: now also U2.4 (I/O2); no longer U2.6 (I/O1)
Changed lines of the file:
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@@
 	(wire
 		(pts
-			(xy 132.08 80.01) (xy 132.08 71.12)
+			(xy 132.08 71.12) (xy 132.08 85.09)
 		)
 		(stroke
@@
 	(wire
 		(pts
+			(xy 128.27 129.54) (xy 128.27 142.24)
+		)
+		(stroke
+			(width 0)
+			(type default)
+		)
+	)
+	(wire
+		(pts
 			(xy 100.33 180.34) (xy 100.33 172.72)
 		)
@@
 	(wire
 		(pts
-			(xy 137.16 80.01) (xy 132.08 80.01)
-		)
-		(stroke
-			(width 0)
-			(type default)
-		)
-	)
-	(wire
-		(pts
 			(xy 38.1 92.71) (xy 101.6 92.71)
 		)
@@
 	(wire
 		(pts
+			(xy 137.16 85.09) (xy 132.08 85.09)
+		)
+		(stroke
+			(width 0)
+			(type default)
+		)
+	)
+	(wire
+		(pts
 			(xy 35.56 31.75) (xy 36.83 31.75)
 		)
@@
 	(wire
 		(pts
-			(xy 101.6 142.24) (xy 124.46 142.24)
+			(xy 101.6 142.24) (xy 128.27 142.24)
 		)
 		(stroke
@@
 	(wire
 		(pts
-			(xy 132.08 85.09) (xy 132.08 92.71)
+			(xy 128.27 129.54) (xy 130.81 129.54)
 		)
 		(stroke
@@
 	(wire
 		(pts
-			(xy 121.92 58.42) (xy 123.19 58.42)
+			(xy 135.255 80.01) (xy 135.255 92.71)
 		)
 		(stroke
@@
 	(wire
 		(pts
-			(xy 140.97 58.42) (xy 146.05 58.42)
-		)
-		(stroke
-			(width 0)
-			(type default)
-		)
-	)
-	(wire
-		(pts
-			(xy 52.07 118.11) (xy 48.26 118.11)
+			(xy 121.92 58.42) (xy 123.19 58.42)
 		)
 		(stroke
@@
 	(wire
 		(pts
-			(xy 35.56 128.27) (xy 35.56 137.16)
+			(xy 140.97 58.42) (xy 146.05 58.42)
 		)
 		(stroke
@@
 	(wire
 		(pts
-			(xy 50.8 78.74) (xy 50.8 83.82)
+			(xy 52.07 118.11) (xy 48.26 118.11)
 		)
 		(stroke
@@
 	(wire
 		(pts
-			(xy 124.46 129.54) (xy 124.46 119.38)
+			(xy 35.56 128.27) (xy 35.56 137.16)
 		)
 		(stroke
@@
 	(wire
 		(pts
-			(xy 124.46 142.24) (xy 124.46 134.62)
+			(xy 50.8 78.74) (xy 50.8 83.82)
 		)
 		(stroke
@@
 	(wire
 		(pts
-			(xy 60.96 162.56) (xy 60.96 160.02)
+			(xy 130.81 134.62) (xy 124.46 134.62)
 		)
 		(stroke
@@
 	(wire
 		(pts
-			(xy 34.29 142.24) (xy 96.52 142.24)
+			(xy 60.96 162.56) (xy 60.96 160.02)
 		)
 		(stroke
@@
 	(wire
 		(pts
-			(xy 234.95 125.73) (xy 232.41 125.73)
+			(xy 34.29 142.24) (xy 96.52 142.24)
 		)
 		(stroke
@@
 	(wire
 		(pts
-			(xy 121.92 66.04) (xy 146.05 66.04)
+			(xy 234.95 125.73) (xy 232.41 125.73)
 		)
 		(stroke
@@
 	(wire
 		(pts
-			(xy 96.52 118.11) (xy 96.52 121.92)
+			(xy 121.92 66.04) (xy 146.05 66.04)
 		)
 		(stroke
@@
 	(wire
 		(pts
-			(xy 137.16 85.09) (xy 132.08 85.09)
+			(xy 96.52 118.11) (xy 96.52 121.92)
 		)
 		(stroke
@@
 	(wire
 		(pts
-			(xy 130.81 129.54) (xy 124.46 129.54)
+			(xy 166.37 162.56) (xy 166.37 160.02)
 		)
 		(stroke
@@
 	(wire
 		(pts
-			(xy 166.37 162.56) (xy 166.37 160.02)
+			(xy 147.32 85.09) (xy 153.67 85.09)
 		)
 		(stroke
@@
 	(wire
 		(pts
-			(xy 147.32 85.09) (xy 153.67 85.09)
+			(xy 33.02 31.75) (xy 35.56 31.75)
 		)
 		(stroke
@@
 	(wire
 		(pts
-			(xy 33.02 31.75) (xy 35.56 31.75)
+			(xy 74.93 95.25) (xy 38.1 95.25)
 		)
 		(stroke
@@
 	(wire
 		(pts
-			(xy 74.93 95.25) (xy 38.1 95.25)
+			(xy 124.46 119.38) (xy 124.46 134.62)
 		)
 		(stroke
@@
 	(wire
 		(pts
-			(xy 124.46 134.62) (xy 130.81 134.62)
+			(xy 137.16 80.01) (xy 135.255 80.01)
 		)
 		(stroke
@@
 	(wire
 		(pts
-			(xy 106.68 92.71) (xy 132.08 92.71)
+			(xy 106.68 92.71) (xy 135.255 92.71)
 		)
 		(stroke
@@
 		)
 	)
+	(label "USB2-DM-ToPad"
+		(at 51.435 139.7 0)
+		(effects
+			(font
+				(size 1.27 1.27)
+			)
+			(justify left bottom)
+		)
+	)
+	(label "USB1-DP-ToPad"
+		(at 53.975 92.71 0)
+		(effects
+			(font
+				(size 1.27 1.27)
+			)
+			(justify left bottom)
+		)
+	)
 	(label "ETH-RXP"
 		(at 147.32 160.02 0)
@@
 		)
 	)
+	(label "USB2-DP-ToESD"
+		(at 109.855 142.24 0)
+		(effects
+			(font
+				(size 1.27 1.27)
+			)
+			(justify left bottom)
+		)
+	)
 	(label "ETH-TXN"
 		(at 62.23 165.1 180)
@@
 		)
 	)
+	(label "USB1-DP-ToESD"
+		(at 117.475 92.71 0)
+		(effects
+			(font
+				(size 1.27 1.27)
+			)
+			(justify left bottom)
+		)
+	)
 	(label "ETH-RXN"
 		(at 147.32 162.56 0)
@@
 		)
 	)
+	(label "USB2-DP-ToPad"
+		(at 51.435 142.24 0)
+		(effects
+			(font
+				(size 1.27 1.27)
+			)
+			(justify left bottom)
+		)
+	)
+	(label "USB1-DM-ToPad"
+		(at 53.975 90.17 0)
+		(effects
+			(font
+				(size 1.27 1.27)
+			)
+			(justify left bottom)
+		)
+	)
+	(label "USB1-DM-ToESD"
+		(at 113.665 71.12 0)
+		(effects
+			(font
+				(size 1.27 1.27)
+			)
+			(justify left bottom)
+		)
+	)
+	(label "USB2-DM-ToESD"
+		(at 105.41 119.38 0)
+		(effects
+			(font
+				(size 1.27 1.27)
+			)
+			(justify left bottom)
+		)
+	)
 	(global_label "VBUS_IN"
 		(shape input)
@@
 	(global_label "USBHost-DM1"
 		(shape input)
-		(at 153.67 80.01 0)
+		(at 153.67 85.09 0)
 		(fields_autoplaced yes)
 		(effects
@@
 		)
 		(property "Intersheetrefs" "${INTERSHEET_REFS}"
-			(at 173.5078 80.01 0)
+			(at 173.5078 85.09 0)
 			(hide yes)
 			(show_name no)
@@
 	(global_label "USBHost-DP2"
 		(shape input)
-		(at 146.05 134.62 0)
+		(at 146.05 129.54 0)
 		(fields_autoplaced yes)
 		(effects
@@
 		)
 		(property "Intersheetrefs" "${INTERSHEET_REFS}"
-			(at 165.6701 134.62 0)
+			(at 165.6701 129.54 0)
 			(hide yes)
 			(show_name no)
@@
 	(global_label "USBHost-DP1"
 		(shape input)
-		(at 153.67 85.09 0)
+		(at 153.67 80.01 0)
 		(fields_autoplaced yes)
 		(effects
@@
 		)
 		(property "Intersheetrefs" "${INTERSHEET_REFS}"
-			(at 173.2901 85.09 0)
+			(at 173.2901 80.01 0)
 			(hide yes)
 			(show_name no)
@@
 	(global_label "USBHost-DM2"
 		(shape input)
-		(at 146.05 129.54 0)
+		(at 146.05 134.62 0)
 		(fields_autoplaced yes)
 		(effects
@@
 		)
 		(property "Intersheetrefs" "${INTERSHEET_REFS}"
-			(at 165.8878 129.54 0)
+			(at 165.8878 134.62 0)
 			(hide yes)
 			(show_name no)
@@
 			)
 		)
-		(property "Description" ""
+		(property "Description" "Unpolarized capacitor"
 			(at 238.76 125.73 0)
 			(hide yes)
@@
 			)
 		)
-		(property "LCSC Part #" "C307331"
+		(property "LCSC Part #" "C1525"
 			(at 186.69 109.22 0)
 			(hide yes)
@@
 			)
 		)
-		(property "LCSC" "C307331"
+		(property "LCSC" "C1525"
 			(at 186.69 109.22 0)
 			(hide yes)
